File: Case/kicad files for case/middle/unisplit_middle.kicad_pcb (KiCad board)
At the start: 2 copper layers, 260.4 x 88.9 mm, 0 parts

Commit message: make case/sleeve fit exactly the same as the pcb, no tolerances
Other:
- board size 260.4 x 88.9 mm -> 254 x 82.6 mm
Changed lines of the file:
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@@
   (general
     (thickness 1.6)
-    (drawings 40)
+    (drawings 36)
     (tracks 0)
     (zones 0)
@@
     (uvia_drill 0.1)
   )
-  (gr_line (start 273.446875 59.928125) (end 153.19375 59.928125) (layer Edge.Cuts) (width 0.05))
-  (gr_line (start 153.19375 53.975) (end 273.05 53.975) (layer Edge.Cuts) (width 0.05))
-  (gr_line (start 29.765625 59.928125) (end 130.96875 59.928125) (layer Edge.Cuts) (width 0.05))
-  (gr_line (start 130.96875 53.975) (end 30.1625 53.975) (layer Edge.Cuts) (width 0.05))
-  (gr_line (start 151.60625 55.5625) (end 151.60625 58.340625) (layer Edge.Cuts) (width 0.05))
-  (gr_line (start 132.55625 55.5625) (end 132.55625 58.340625) (layer Edge.Cuts) (width 0.05))
-  (gr_arc (start 130.96875 58.340625) (end 130.96875 59.928125) (angle -90) (layer Edge.Cuts) (width 0.05))
-  (gr_arc (start 153.19375 55.5625) (end 153.19375 53.975) (angle -90) (layer Edge.Cuts) (width 0.05))
-  (gr_arc (start 153.19375 58.340625) (end 151.60625 58.340625) (angle -90) (layer Edge.Cuts) (width 0.05))
-  (gr_arc (start 130.96875 55.5625) (end 132.55625 55.5625) (angle -90) (layer Edge.Cuts) (width 0.05))
-  (gr_arc (start 227.0125 107.15625) (end 227.0125 104.775) (angle -90) (layer Edge.Cuts) (width 0.05))
-  (gr_line (start 21.43125 62.70625) (end 21.43125 96.04375) (layer Edge.Cuts) (width 0.05))
-  (gr_line (start 224.63125 134.14375) (end 224.63125 107.15625) (layer Edge.Cuts) (width 0.05))
-  (gr_line (start 68.2625 142.875) (end 215.9 142.875) (layer Edge.Cuts) (width 0.05))
-  (gr_arc (start 57.15 107.15625) (end 59.53125 107.15625) (angle -90) (layer Edge.Cuts) (width 0.05))
-  (gr_line (start 59.53125 107.15625) (end 59.53125 134.14375) (layer Edge.Cuts) (width 0.05))
-  (gr_line (start 281.78125 96.04375) (end 281.78125 62.70625) (layer Edge.Cuts) (width 0.05))
-  (gr_line (start 227.0125 104.775) (end 273.05 104.775) (layer Edge.Cuts) (width 0.05))
-  (gr_arc (start 273.05 62.70625) (end 281.78125 62.70625) (angle -90) (layer Edge.Cuts) (width 0.05))
-  (gr_arc (start 68.2625 134.14375) (end 59.53125 134.14375) (angle -90) (layer Edge.Cuts) (width 0.05))
-  (gr_line (start 57.15 104.775) (end 30.1625 104.775) (layer Edge.Cuts) (width 0.05))
-  (gr_arc (start 30.1625 62.70625) (end 30.1625 53.975) (angle -90) (layer Edge.Cuts) (width 0.05))
-  (gr_arc (start 30.1625 96.04375) (end 21.43125 96.04375) (angle -90) (layer Edge.Cuts) (width 0.05))
-  (gr_arc (start 215.9 134.14375) (end 215.9 142.875) (angle -90) (layer Edge.Cuts) (width 0.05))
-  (gr_arc (start 273.05 96.04375) (end 273.05 104.775) (angle -90) (layer Edge.Cuts) (width 0.05))
-  (gr_line (start 221.059375 98.821875) (end 273.446875 98.821875) (layer Edge.Cuts) (width 0.05))
-  (gr_line (start 218.678125 134.540625) (end 218.678125 101.203125) (layer Edge.Cuts) (width 0.05))
-  (gr_line (start 67.865625 136.921875) (end 216.296875 136.921875) (layer Edge.Cuts) (width 0.05))
-  (gr_line (start 65.484375 101.203125) (end 65.484375 134.540625) (layer Edge.Cuts) (width 0.05))
-  (gr_line (start 29.765625 98.821875) (end 63.103125 98.821875) (layer Edge.Cuts) (width 0.05))
-  (gr_arc (start 67.865625 134.540625) (end 65.484375 134.540625) (angle -90) (layer Edge.Cuts) (width 0.05))
-  (gr_arc (start 216.296875 134.540625) (end 216.296875 136.921875) (angle -90) (layer Edge.Cuts) (width 0.05))
-  (gr_arc (start 221.059375 101.203125) (end 221.059375 98.821875) (angle -90) (layer Edge.Cuts) (width 0.05))
-  (gr_arc (start 63.103125 101.203125) (end 65.484375 101.203125) (angle -90) (layer Edge.Cuts) (width 0.05))
-  (gr_line (start 275.828125 96.440625) (end 275.828125 62.309375) (layer Edge.Cuts) (width 0.05))
-  (gr_line (start 27.384375 62.309375) (end 27.384375 96.440625) (layer Edge.Cuts) (width 0.05))
-  (gr_arc (start 29.765625 62.309375) (end 29.765625 59.928125) (angle -90) (layer Edge.Cuts) (width 0.05))
-  (gr_arc (start 29.765625 96.440625) (end 27.384375 96.440625) (angle -90) (layer Edge.Cuts) (width 0.05))
-  (gr_arc (start 273.446875 96.440625) (end 273.446875 98.821875) (angle -90) (layer Edge.Cuts) (width 0.05))
-  (gr_arc (start 273.446875 62.309375) (end 275.828125 62.309375) (angle -90) (layer Edge.Cuts) (width 0.05))
+  (gr_arc (start 215.9 134.14375) (end 215.9 139.7) (angle -90) (layer Edge.Cuts) (width 0.05))
+  (gr_line (start 273.05 60.325) (end 153.19375 60.325) (layer Edge.Cuts) (width 0.05))
+  (gr_line (start 153.19375 57.15) (end 273.05 57.15) (layer Edge.Cuts) (width 0.05))
+  (gr_line (start 30.1625 60.325) (end 130.96875 60.325) (layer Edge.Cuts) (width 0.05))
+  (gr_line (start 130.96875 57.15) (end 30.1625 57.15) (layer Edge.Cuts) (width 0.05))
+  (gr_arc (start 130.96875 58.7375) (end 130.96875 60.325) (angle -180) (layer Edge.Cuts) (width 0.05))
+  (gr_arc (start 153.19375 58.7375) (end 153.19375 57.15) (angle -180) (layer Edge.Cuts) (width 0.05))
+  (gr_arc (start 223.8375 103.98125) (end 223.8375 101.6) (angle -90) (layer Edge.Cuts) (width 0.05))
+  (gr_line (start 24.60625 62.70625) (end 24.60625 96.04375) (layer Edge.Cuts) (width 0.05))
+  (gr_line (start 221.45625 134.14375) (end 221.45625 103.98125) (layer Edge.Cuts) (width 0.05))
+  (gr_line (start 68.2625 139.7) (end 215.9 139.7) (layer Edge.Cuts) (width 0.05))
+  (gr_arc (start 60.325 103.98125) (end 62.70625 103.98125) (angle -90) (layer Edge.Cuts) (width 0.05))
+  (gr_line (start 62.70625 103.98125) (end 62.70625 134.14375) (layer Edge.Cuts) (width 0.05))
+  (gr_line (start 278.60625 96.04375) (end 278.60625 62.70625) (layer Edge.Cuts) (width 0.05))
+  (gr_line (start 223.8375 101.6) (end 273.05 101.6) (layer Edge.Cuts) (width 0.05))
+  (gr_arc (start 273.05 62.70625) (end 278.60625 62.70625) (angle -90) (layer Edge.Cuts) (width 0.05))
+  (gr_arc (start 68.2625 134.14375) (end 62.70625 134.14375) (angle -90) (layer Edge.Cuts) (width 0.05))
+  (gr_line (start 60.325 101.6) (end 30.1625 101.6) (layer Edge.Cuts) (width 0.05))
+  (gr_arc (start 30.1625 62.70625) (end 30.1625 57.15) (angle -90) (layer Edge.Cuts) (width 0.05))
+  (gr_arc (start 30.1625 96.04375) (end 24.60625 96.04375) (angle -90) (layer Edge.Cuts) (width 0.05))
+  (gr_arc (start 273.05 96.04375) (end 273.05 101.6) (angle -90) (layer Edge.Cuts) (width 0.05))
+  (gr_line (start 220.6625 98.425) (end 273.05 98.425) (layer Edge.Cuts) (width 0.05))
+  (gr_line (start 218.28125 134.14375) (end 218.28125 100.80625) (layer Edge.Cuts) (width 0.05))
+  (gr_line (start 68.2625 136.525) (end 215.9 136.525) (layer Edge.Cuts) (width 0.05))
+  (gr_line (start 65.88125 100.80625) (end 65.88125 134.14375) (layer Edge.Cuts) (width 0.05))
+  (gr_line (start 30.1625 98.425) (end 63.5 98.425) (layer Edge.Cuts) (width 0.05))
+  (gr_arc (start 68.2625 134.14375) (end 65.88125 134.14375) (angle -90) (layer Edge.Cuts) (width 0.05))
+  (gr_arc (start 215.9 134.14375) (end 215.9 136.525) (angle -90) (layer Edge.Cuts) (width 0.05))
+  (gr_arc (start 220.6625 100.80625) (end 220.6625 98.425) (angle -90) (layer Edge.Cuts) (width 0.05))
+  (gr_arc (start 63.5 100.80625) (end 65.88125 100.80625) (angle -90) (layer Edge.Cuts) (width 0.05))
+  (gr_line (start 275.43125 96.04375) (end 275.43125 62.70625) (layer Edge.Cuts) (width 0.05))
+  (gr_line (start 27.78125 62.70625) (end 27.78125 96.04375) (layer Edge.Cuts) (width 0.05))
+  (gr_arc (start 30.1625 62.70625) (end 30.1625 60.325) (angle -90) (layer Edge.Cuts) (width 0.05))
+  (gr_arc (start 30.1625 96.04375) (end 27.78125 96.04375) (angle -90) (layer Edge.Cuts) (width 0.05))
+  (gr_arc (start 273.05 96.04375) (end 273.05 98.425) (angle -90) (layer Edge.Cuts) (width 0.05))
+  (gr_arc (start 273.05 62.70625) (end 275.43125 62.70625) (angle -90) (layer Edge.Cuts) (width 0.05))
 )
