File: Case/kicad files for case/bottom/unisplit_bottom.kicad_pcb (KiCad board)
At the start: 2 copper layers, 255.6 x 84.1 mm, 0 parts

Commit message: update case files by giving a little bit of clearance
Other:
- board size 255.6 x 84.1 mm -> 260.4 x 88.9 mm

Commit message: make case/sleeve fit exactly the same as the pcb, no tolerances
Other:
- board size 260.4 x 88.9 mm -> 254 x 82.6 mm
Changed lines of the file:
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@@
     (uvia_drill 0.1)
   )
-  (gr_line (start 21.43125 62.70625) (end 21.43125 96.04375) (layer Edge.Cuts) (width 0.05))
-  (gr_line (start 273.05 53.975) (end 30.1625 53.975) (layer Edge.Cuts) (width 0.05))
-  (gr_line (start 281.78125 96.04375) (end 281.78125 62.70625) (layer Edge.Cuts) (width 0.05))
-  (gr_line (start 227.0125 104.775) (end 273.05 104.775) (layer Edge.Cuts) (width 0.05))
-  (gr_line (start 224.63125 134.14375) (end 224.63125 107.15625) (layer Edge.Cuts) (width 0.05))
-  (gr_line (start 68.2625 142.875) (end 215.9 142.875) (layer Edge.Cuts) (width 0.05))
-  (gr_line (start 57.15 104.775) (end 30.1625 104.775) (layer Edge.Cuts) (width 0.05))
-  (gr_line (start 59.53125 107.15625) (end 59.53125 134.14375) (layer Edge.Cuts) (width 0.05))
-  (gr_arc (start 57.15 107.15625) (end 59.53125 107.15625) (angle -90) (layer Edge.Cuts) (width 0.05))
-  (gr_arc (start 227.0125 107.15625) (end 227.0125 104.775) (angle -90) (layer Edge.Cuts) (width 0.05))
-  (gr_arc (start 68.2625 134.14375) (end 59.53125 134.14375) (angle -90) (layer Edge.Cuts) (width 0.05))
-  (gr_arc (start 30.1625 96.04375) (end 21.43125 96.04375) (angle -90) (layer Edge.Cuts) (width 0.05))
-  (gr_arc (start 30.1625 62.70625) (end 30.1625 53.975) (angle -90) (layer Edge.Cuts) (width 0.05))
-  (gr_arc (start 273.05 62.70625) (end 281.78125 62.70625) (angle -90) (layer Edge.Cuts) (width 0.05))
-  (gr_arc (start 273.05 96.04375) (end 273.05 104.775) (angle -90) (layer Edge.Cuts) (width 0.05))
-  (gr_arc (start 215.9 134.14375) (end 215.9 142.875) (angle -90) (layer Edge.Cuts) (width 0.05))
+  (gr_arc (start 215.9 134.14375) (end 215.9 139.7) (angle -90) (layer Edge.Cuts) (width 0.05))
+  (gr_line (start 273.05 57.15) (end 30.1625 57.15) (layer Edge.Cuts) (width 0.05))
+  (gr_arc (start 223.8375 103.98125) (end 223.8375 101.6) (angle -90) (layer Edge.Cuts) (width 0.05))
+  (gr_line (start 24.60625 62.70625) (end 24.60625 96.04375) (layer Edge.Cuts) (width 0.05))
+  (gr_line (start 221.45625 134.14375) (end 221.45625 103.98125) (layer Edge.Cuts) (width 0.05))
+  (gr_line (start 68.2625 139.7) (end 215.9 139.7) (layer Edge.Cuts) (width 0.05))
+  (gr_arc (start 60.325 103.98125) (end 62.70625 103.98125) (angle -90) (layer Edge.Cuts) (width 0.05))
+  (gr_line (start 62.70625 103.98125) (end 62.70625 134.14375) (layer Edge.Cuts) (width 0.05))
+  (gr_line (start 278.60625 96.04375) (end 278.60625 62.70625) (layer Edge.Cuts) (width 0.05))
+  (gr_line (start 223.8375 101.6) (end 273.05 101.6) (layer Edge.Cuts) (width 0.05))
+  (gr_arc (start 273.05 62.70625) (end 278.60625 62.70625) (angle -90) (layer Edge.Cuts) (width 0.05))
+  (gr_arc (start 68.2625 134.14375) (end 62.70625 134.14375) (angle -90) (layer Edge.Cuts) (width 0.05))
+  (gr_line (start 60.325 101.6) (end 30.1625 101.6) (layer Edge.Cuts) (width 0.05))
+  (gr_arc (start 30.1625 62.70625) (end 30.1625 57.15) (angle -90) (layer Edge.Cuts) (width 0.05))
+  (gr_arc (start 30.1625 96.04375) (end 24.60625 96.04375) (angle -90) (layer Edge.Cuts) (width 0.05))
+  (gr_arc (start 273.05 96.04375) (end 273.05 101.6) (angle -90) (layer Edge.Cuts) (width 0.05))
 )
