File: Case/kicad files for case/actual size of pcb/unisplit_orthosteno.kicad_pcb (KiCad board)
At the start: 2 copper layers, 254 x 82.6 mm, 0 parts

Commit message: add split case files for easy printing
Other:
- board size 254 x 82.6 mm -> 247.6 x 76.2 mm
Changed lines of the file:
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@@
   (general
     (thickness 1.6)
-    (drawings 36)
+    (drawings 20)
     (tracks 0)
     (zones 0)
@@
     (uvia_drill 0.1)
   )
-  (gr_arc (start 215.9 134.14375) (end 215.9 139.7) (angle -90) (layer Edge.Cuts) (width 0.05))
-  (gr_line (start 273.05 60.325) (end 153.19375 60.325) (layer Edge.Cuts) (width 0.05))
-  (gr_line (start 153.19375 57.15) (end 273.05 57.15) (layer Edge.Cuts) (width 0.05))
-  (gr_line (start 30.1625 60.325) (end 130.96875 60.325) (layer Edge.Cuts) (width 0.05))
-  (gr_line (start 130.96875 57.15) (end 30.1625 57.15) (layer Edge.Cuts) (width 0.05))
-  (gr_arc (start 130.96875 58.7375) (end 130.96875 60.325) (angle -180) (layer Edge.Cuts) (width 0.05))
-  (gr_arc (start 153.19375 58.7375) (end 153.19375 57.15) (angle -180) (layer Edge.Cuts) (width 0.05))
-  (gr_arc (start 223.8375 103.98125) (end 223.8375 101.6) (angle -90) (layer Edge.Cuts) (width 0.05))
-  (gr_line (start 24.60625 62.70625) (end 24.60625 96.04375) (layer Edge.Cuts) (width 0.05))
-  (gr_line (start 221.45625 134.14375) (end 221.45625 103.98125) (layer Edge.Cuts) (width 0.05))
-  (gr_line (start 68.2625 139.7) (end 215.9 139.7) (layer Edge.Cuts) (width 0.05))
-  (gr_arc (start 60.325 103.98125) (end 62.70625 103.98125) (angle -90) (layer Edge.Cuts) (width 0.05))
-  (gr_line (start 62.70625 103.98125) (end 62.70625 134.14375) (layer Edge.Cuts) (width 0.05))
-  (gr_line (start 278.60625 96.04375) (end 278.60625 62.70625) (layer Edge.Cuts) (width 0.05))
-  (gr_line (start 223.8375 101.6) (end 273.05 101.6) (layer Edge.Cuts) (width 0.05))
-  (gr_arc (start 273.05 62.70625) (end 278.60625 62.70625) (angle -90) (layer Edge.Cuts) (width 0.05))
-  (gr_arc (start 68.2625 134.14375) (end 62.70625 134.14375) (angle -90) (layer Edge.Cuts) (width 0.05))
-  (gr_line (start 60.325 101.6) (end 30.1625 101.6) (layer Edge.Cuts) (width 0.05))
-  (gr_arc (start 30.1625 62.70625) (end 30.1625 57.15) (angle -90) (layer Edge.Cuts) (width 0.05))
-  (gr_arc (start 30.1625 96.04375) (end 24.60625 96.04375) (angle -90) (layer Edge.Cuts) (width 0.05))
-  (gr_arc (start 273.05 96.04375) (end 273.05 101.6) (angle -90) (layer Edge.Cuts) (width 0.05))
+  (gr_line (start 132.55625 60.325) (end 30.1625 60.325) (layer Edge.Cuts) (width 0.05))
+  (gr_line (start 151.60625 60.325) (end 273.05 60.325) (layer Edge.Cuts) (width 0.05))
+  (gr_line (start 151.60625 63.5) (end 151.60625 60.325) (layer Edge.Cuts) (width 0.05))
+  (gr_line (start 132.55625 60.325) (end 151.60625 60.325) (layer Edge.Cuts) (width 0.05))
+  (gr_line (start 132.55625 60.325) (end 132.55625 63.5) (layer Edge.Cuts) (width 0.05))
   (gr_line (start 220.6625 98.425) (end 273.05 98.425) (layer Edge.Cuts) (width 0.05))
   (gr_line (start 218.28125 134.14375) (end 218.28125 100.80625) (layer Edge.Cuts) (width 0.05))
