File: Case/kicad files for case/back-plate/back-plate.kicad_pcb (KiCad board)
At the start: 2 copper layers, 247.6 x 76.2 mm, 6 parts

Commit message: backplate design
Parts:
- added Ref**: Val**, library:full-graphic, F.Cu at (149.9, 85.2)
