File: Case/kicad files for case/back-plate/back-plate.kicad_pcb (KiCad board)
At the start: 2 copper layers, 247.6 x 76.2 mm, 7 parts

Commit message: add rubber feet placement image
Routing:
- added copper zone on B.Cu, net (none)
- added copper zone on F.Cu, net (none)

Commit message: save backplate file
Other:
- net class Default removed
