File: unisplit_orthosteno.kicad_pcb (KiCad board)
At the start: 2 copper layers, 53 parts, among them U1 ProMicro

Commit message: finished routing but possible problem in column 3 and 4 which I asked and reddit
Parts:
- added D25: SOD-123, Keebio-Parts:D_SOD123, B.Cu at (142.1, 131.8)
- added MX25: MX-NoLED, Keebio-Parts:MX-Alps-Choc-1U-NoLED, F.Cu at (142.1, 127.0)
- moved D22 185.8 mm to (265.9, 93.7)
- moved D11 185.6 mm to (265.9, 74.6)
- moved D10 160.8 mm to (246.9, 74.6)
- moved D21 159.5 mm to (246.9, 93.7)
- moved D1 151.6 mm to (37.3, 74.6)
- moved D12 145.6 mm to (37.3, 93.7)
- moved D9 137.0 mm to (227.8, 74.6)
- moved D20 134.6 mm to (227.8, 93.7)
- moved D2 127.7 mm to (56.4, 74.6)
- moved D13 120.4 mm to (56.4, 93.7)
- moved D8 114.5 mm to (208.8, 74.6)
- moved D19 111.3 mm to (208.8, 93.7)
- moved U1 109.4 mm to (142.1, 77.8)
- moved D3 106.4 mm to (75.3, 74.6)
- moved D14 97.5 mm to (75.4, 93.7)
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- renumbered D25 to D26, D26 to D27, MX25 to MX26, MX26 to MX27
Connections:
- MX23 pad 1: col3 -> col2
- MX24 pad 1: col4 -> col3
- U1 pad 13: row0 -> row2
- U1 pad 14: row1 -> row0
- U1 pad 15: row2 -> row1
- U1 pad 16: col0 -> col4
- U1 pad 17: col1 -> col3
- U1 pad 19: col3 -> col1
- U1 pad 20: col4 -> col0
Routing:
- net row0: track 0.00 -> 368.1 mm, vias 0 -> 2
- net row1: track 0.00 -> 337.6 mm, vias 0 -> 2
- net row2: track 0.00 -> 155.0 mm
- net col10: track 0.00 -> 146.4 mm
- net col2: track 0.00 -> 129.5 mm
- net col9: track 0.00 -> 126.7 mm
- net col6: track 0.00 -> 122.6 mm
- net col0: track 0.00 -> 121.7 mm
- net col8: track 0.00 -> 108.9 mm
- net col3: track 0.00 -> 108.8 mm
- net col5: track 0.00 -> 106.5 mm
- net col1: track 0.00 -> 101.6 mm
- net col4: track 0.00 -> 92.0 mm
- net col7: track 0.00 -> 90.3 mm
- net Net-(D8-Pad2): track 0.00 -> 13.4 mm
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
Commit message: re route and change layout per suggestions from plover discord
Parts:
- added D28: SOD-123, Keebio-Parts:D_SOD123, B.Cu at (208.8, 131.8)
- added MX28: MX-NoLED, Keebio-Parts:MX-Alps-Choc-1U-NoLED, F.Cu at (208.8, 127.0)
- moved D25 28.6 mm to (113.5, 131.8)
- moved MX25 28.6 mm to (113.5, 127.0)
- moved D23 19.0 mm to (75.4, 131.8)
- moved D24 19.0 mm to (94.5, 131.8)
- moved MX23 19.0 mm to (75.4, 127.0)
- moved MX24 19.0 mm to (94.5, 127.0)
Connections:
- net Net-(U1-Pad21) renamed +5V
- U1 pad 14: row0 -> row1
- U1 pad 15: row1 -> col4
- U1 pad 16: col4 -> col3
- U1 pad 17: col3 -> col2
- U1 pad 18: col2 -> col1
- U1 pad 19: col1 -> col0
- U1 pad 20: col0 -> row0
- U1 pad 23: Net-(U1-Pad23) -> GND
- U1 pad 3: Net-(U1-Pad3) -> GND
- U1 pad 4: Net-(U1-Pad4) -> GND
Routing:
- net row0: track 368.1 -> 237.6 mm, vias 2 -> 0
- net row1: track 337.6 -> 240.8 mm, vias 2 -> 0
- net col7: track 90.3 -> 131.6 mm
- net row2: track 155.0 -> 177.7 mm
- net GND: track 0.00 -> 18.8 mm
- net col5: track 106.5 -> 94.9 mm
- net Net-(D28-Pad2): track 0.00 -> 11.5 mm
- net col6: track 122.6 -> 113.2 mm
- net col2: track 129.5 -> 123.9 mm
- net col4: track 92.0 -> 88.3 mm
- net col3: track 108.8 -> 105.6 mm
- net Net-(D8-Pad2): track 13.4 -> 11.5 mm
- net Net-(D9-Pad2): track 11.5 -> 13.4 mm
- net Net-(D7-Pad2): track 13.4 -> 11.5 mm
- net Net-(D6-Pad2): track 11.5 -> 13.4 mm
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Other:
- board outline added: 247.6 x 76.2 mm

Commit message: generate gerbers
Routing:
- net GND: track 18.8 -> 16.3 mm
- added copper zone on B.Cu, net GND
- added copper zone on F.Cu, net GND
Other:
- board text added: "Peter C. Park Design"
Changed lines of the file:
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@@
   (general
     (thickness 1.6)
-    (drawings 356)
-    (tracks 350)
+    (drawings 357)
+    (tracks 349)
     (zones 0)
     (modules 57)
@@
     (pcbplotparams
       (layerselection 0x010fc_ffffffff)
-      (usegerberextensions false)
+      (usegerberextensions true)
       (usegerberattributes true)
       (usegerberadvancedattributes true)
@@
       (outputformat 1)
       (mirror false)
-      (drillshape 1)
+      (drillshape 0)
       (scaleselection 1)
-      (outputdirectory ""))
+      (outputdirectory "Gerbers/"))
   )
   (net 0 "")
@@
     (pad 2 smd rect (at 1.7 0 180) (size 1.2 1.4) (layers B.Cu B.Paste B.Mask)
       (net 2 "Net-(D1-Pad2)"))
+  )
+  (gr_text "Peter C. Park Design" (at 142.08125 127.79375) (layer F.SilkS)
+    (effects (font (size 2 2) (thickness 0.2)))
   )
   (gr_line (start 220.6625 98.425) (end 273.05 98.425) (layer Edge.Cuts) (width 0.05))
@@
   (segment (start 147.16125 66.3575) (end 149.70125 68.8975) (width 0.25) (layer B.Cu) (net 49))
   (segment (start 134.46125 66.3575) (end 147.16125 66.3575) (width 0.25) (layer B.Cu) (net 49))
-  (segment (start 149.70125 68.8975) (end 149.70125 71.4375) (width 0.25) (layer B.Cu) (net 49))
+  (zone (net 49) (net_name GND) (layer F.Cu) (hatch edge 0.508)
+    (connect_pads (clearance 0.508))
+    (min_thickness 0.254)
+    (fill yes (arc_segments 32) (thermal_gap 0.508) (thermal_bridge_width 0.508))
+    (polygon
+      (pts
+        (xy 275.43125 98.425) (xy 218.28125 98.425) (xy 218.28125 136.525) (xy 65.88125 136.525) (xy 65.88125 98.425)
+        (xy 27.78125 98.425) (xy 27.78125 60.325) (xy 275.43125 60.325)
+      )
+    )
+  )
+  (zone (net 49) (net_name GND) (layer B.Cu) (hatch edge 0.508)
+    (connect_pads (clearance 0.508))
+    (min_thickness 0.254)
+    (fill yes (arc_segments 32) (thermal_gap 0.508) (thermal_bridge_width 0.508))
+    (polygon
+      (pts
+        (xy 275.43125 98.425) (xy 218.28125 98.425) (xy 218.28125 136.525) (xy 65.88125 136.525) (xy 65.88125 98.425)
+        (xy 27.78125 98.425) (xy 27.78125 60.325) (xy 275.43125 60.325)
+      )
+    )
+  )
 )

Commit message: finalize gerbers and create bom and place files for jlcpcb
Connections:
- net +5V renamed Net-(U1-Pad21)
Changed lines of the file:
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@@
     (visible_elements 7FFFFFFF)
     (pcbplotparams
-      (layerselection 0x010fc_ffffffff)
+      (layerselection 0x010f0_ffffffff)
       (usegerberextensions true)
-      (usegerberattributes true)
-      (usegerberadvancedattributes true)
-      (creategerberjobfile true)
+      (usegerberattributes false)
+      (usegerberadvancedattributes false)
+      (creategerberjobfile false)
       (excludeedgelayer true)
       (linewidth 0.100000)
@@
       (plotinvisibletext false)
       (padsonsilk false)
-      (subtractmaskfromsilk false)
+      (subtractmaskfromsilk true)
       (outputformat 1)
       (mirror false)
@@
   (net 41 "Net-(U1-Pad24)")
   (net 42 "Net-(U1-Pad22)")
-  (net 43 "Net-(U1-Pad2)")
-  (net 44 "Net-(U1-Pad1)")
-  (net 45 "Net-(U1-Pad6)")
-  (net 46 "Net-(U1-Pad5)")
-  (net 47 "Net-(D27-Pad2)")
-  (net 48 "Net-(D28-Pad2)")
-  (net 49 GND)
-  (net 50 +5V)
+  (net 43 "Net-(U1-Pad21)")
+  (net 44 "Net-(U1-Pad2)")
+  (net 45 "Net-(U1-Pad1)")
+  (net 46 "Net-(U1-Pad6)")
+  (net 47 "Net-(U1-Pad5)")
+  (net 48 "Net-(D27-Pad2)")
+  (net 49 "Net-(D28-Pad2)")
+  (net 50 GND)
   (net_class Default "This is the default net class."
     (clearance 0.2)
@@
     (uvia_dia 0.3)
     (uvia_drill 0.1)
-    (add_net +5V)
     (add_net GND)
     (add_net "Net-(D1-Pad2)")
@@
     (add_net "Net-(U1-Pad1)")
     (add_net "Net-(U1-Pad2)")
+    (add_net "Net-(U1-Pad21)")
     (add_net "Net-(U1-Pad22)")
     (add_net "Net-(U1-Pad24)")
@@
     (pad "" np_thru_hole circle (at -5.5 0 48.1) (size 1.7 1.7) (drill 1.7) (layers *.Cu *.Mask))
     (pad 2 thru_hole circle (at 0 -5.9) (size 2 2) (drill 1.2) (layers *.Cu *.Mask)
-      (net 48 "Net-(D28-Pad2)"))
+      (net 49 "Net-(D28-Pad2)"))
     (pad 1 thru_hole circle (at 5 -3.8) (size 2 2) (drill 1.2) (layers *.Cu *.Mask)
       (net 37 col7))
@@
     (pad "" np_thru_hole circle (at -5.08 0 48.0996) (size 1.75 1.75) (drill 1.75) (layers *.Cu *.Mask))
     (pad 2 thru_hole circle (at -2.5 -4) (size 2.25 2.25) (drill 1.47) (layers *.Cu *.Mask)
-      (net 48 "Net-(D28-Pad2)"))
+      (net 49 "Net-(D28-Pad2)"))
     (pad "" np_thru_hole circle (at 0 0) (size 3.9878 3.9878) (drill 3.9878) (layers *.Cu *.Mask))
     (pad 2 thru_hole oval (at -3.81 -2.54 48.1) (size 4.211556 2.25) (drill 1.47 (offset 0.980778 0)) (layers *.Cu *.Mask)
-      (net 48 "Net-(D28-Pad2)"))
+      (net 49 "Net-(D28-Pad2)"))
     (pad 1 thru_hole circle (at 2.54 -5.08) (size 2.25 2.25) (drill 1.47) (layers *.Cu *.Mask)
       (net 37 col7))
@@
       (net 25 row2))
     (pad 2 smd rect (at 1.7 0 180) (size 1.2 1.4) (layers B.Cu B.Paste B.Mask)
-      (net 48 "Net-(D28-Pad2)"))
+      (net 49 "Net-(D28-Pad2)"))
   )
   (module Keebio-Parts:MX-Alps-Choc-1U-NoLED (layer F.Cu)
@@
       (net 35 col5))
     (pad 23 thru_hole circle (at -11.43 7.62 270) (size 1.7526 1.7526) (drill 1.0922) (layers *.Cu *.SilkS *.Mask)
-      (net 49 GND))
+      (net 50 GND))
     (pad 22 thru_hole circle (at -8.89 7.62 270) (size 1.7526 1.7526) (drill 1.0922) (layers *.Cu *.SilkS *.Mask)
       (net 42 "Net-(U1-Pad22)"))
     (pad 21 thru_hole circle (at -6.35 7.62 270) (size 1.7526 1.7526) (drill 1.0922) (layers *.Cu *.SilkS *.Mask)
-      (net 50 +5V))
+      (net 43 "Net-(U1-Pad21)"))
     (pad 20 thru_hole circle (at -3.81 7.62 270) (size 1.7526 1.7526) (drill 1.0922) (layers *.Cu *.SilkS *.Mask)
       (net 1 row0))
@@
       (net 40 col10))
     (pad 6 thru_hole circle (at -1.27 -7.62 270) (size 1.7526 1.7526) (drill 1.0922) (layers *.Cu *.SilkS *.Mask)
-      (net 45 "Net-(U1-Pad6)"))
+      (net 46 "Net-(U1-Pad6)"))
     (pad 5 thru_hole circle (at -3.81 -7.62 270) (size 1.7526 1.7526) (drill 1.0922) (layers *.Cu *.SilkS *.Mask)
-      (net 46 "Net-(U1-Pad5)"))
+      (net 47 "Net-(U1-Pad5)"))
     (pad 4 thru_hole circle (at -6.35 -7.62 270) (size 1.7526 1.7526) (drill 1.0922) (layers *.Cu *.SilkS *.Mask)
-      (net 49 GND))
+      (net 50 GND))
     (pad 3 thru_hole circle (at -8.89 -7.62 270) (size 1.7526 1.7526) (drill 1.0922) (layers *.Cu *.SilkS *.Mask)
-      (net 49 GND))
+      (net 50 GND))
     (pad 2 thru_hole circle (at -11.43 -7.62 270) (size 1.7526 1.7526) (drill 1.0922) (layers *.Cu *.SilkS *.Mask)
-      (net 43 "Net-(U1-Pad2)"))
+      (net 44 "Net-(U1-Pad2)"))
     (pad 1 thru_hole rect (at -13.97 -7.62 270) (size 1.7526 1.7526) (drill 1.0922) (layers *.Cu *.SilkS *.Mask)
-      (net 44 "Net-(U1-Pad1)"))
+      (net 45 "Net-(U1-Pad1)"))
     (model /Users/danny/Documents/proj/custom-keyboard/kicad-libs/3d_models/ArduinoProMicro.wrl
       (offset (xyz -13.96999979019165 -7.619999885559082 -5.841999912261963))
@@
     (pad "" np_thru_hole circle (at -5.5 0 48.1) (size 1.7 1.7) (drill 1.7) (layers *.Cu *.Mask))
     (pad 2 thru_hole circle (at 0 -5.9) (size 2 2) (drill 1.2) (layers *.Cu *.Mask)
-      (net 47 "Net-(D27-Pad2)"))
+      (net 48 "Net-(D27-Pad2)"))
     (pad 1 thru_hole circle (at 5 -3.8) (size 2 2) (drill 1.2) (layers *.Cu *.Mask)
       (net 36 col6))
@@
     (pad "" np_thru_hole circle (at -5.08 0 48.0996) (size 1.75 1.75) (drill 1.75) (layers *.Cu *.Mask))
     (pad 2 thru_hole circle (at -2.5 -4) (size 2.25 2.25) (drill 1.47) (layers *.Cu *.Mask)
-      (net 47 "Net-(D27-Pad2)"))
+      (net 48 "Net-(D27-Pad2)"))
     (pad "" np_thru_hole circle (at 0 0) (size 3.9878 3.9878) (drill 3.9878) (layers *.Cu *.Mask))
     (pad 2 thru_hole oval (at -3.81 -2.54 48.1) (size 4.211556 2.25) (drill 1.47 (offset 0.980778 0)) (layers *.Cu *.Mask)
-      (net 47 "Net-(D27-Pad2)"))
+      (net 48 "Net-(D27-Pad2)"))
     (pad 1 thru_hole circle (at 2.54 -5.08) (size 2.25 2.25) (drill 1.47) (layers *.Cu *.Mask)
       (net 36 col6))
@@
       (net 25 row2))
     (pad 2 smd rect (at 1.7 0 180) (size 1.2 1.4) (layers B.Cu B.Paste B.Mask)
-      (net 47 "Net-(D27-Pad2)"))
+      (net 48 "Net-(D27-Pad2)"))
   )
   (module Keebio-Parts:D_SOD123 (layer B.Cu)
@@
   (segment (start 268.40625 83.538998) (end 263.924752 79.0575) (width 0.25) (layer B.Cu) (net 40))
   (segment (start 268.40625 84.4) (end 268.40625 83.538998) (width 0.25) (layer B.Cu) (net 40))
-  (segment (start 186.34625 124.46) (end 185.89625 124.46) (width 0.25) (layer B.Cu) (net 47))
-  (segment (start 189.70625 121.1) (end 186.34625 124.46) (width 0.25) (layer B.Cu) (net 47))
-  (segment (start 185.89625 129.6525) (end 188.00625 131.7625) (width 0.25) (layer B.Cu) (net 47))
-  (segment (start 185.89625 124.46) (end 185.89625 129.6525) (width 0.25) (layer B.Cu) (net 47))
-  (segment (start 206.85625 123) (end 206.25625 123) (width 0.25) (layer B.Cu) (net 48))
-  (segment (start 208.75625 121.1) (end 206.85625 123) (width 0.25) (layer B.Cu) (net 48))
-  (segment (start 204.94625 129.6525) (end 207.05625 131.7625) (width 0.25) (layer B.Cu) (net 48))
-  (segment (start 204.94625 124.46) (end 204.94625 129.6525) (width 0.25) (layer B.Cu) (net 48))
-  (segment (start 147.16125 66.3575) (end 149.70125 68.8975) (width 0.25) (layer B.Cu) (net 49))
-  (segment (start 134.46125 66.3575) (end 147.16125 66.3575) (width 0.25) (layer B.Cu) (net 49))
-  (zone (net 49) (net_name GND) (layer F.Cu) (hatch edge 0.508)
+  (segment (start 186.34625 124.46) (end 185.89625 124.46) (width 0.25) (layer B.Cu) (net 48))
+  (segment (start 189.70625 121.1) (end 186.34625 124.46) (width 0.25) (layer B.Cu) (net 48))
+  (segment (start 185.89625 129.6525) (end 188.00625 131.7625) (width 0.25) (layer B.Cu) (net 48))
+  (segment (start 185.89625 124.46) (end 185.89625 129.6525) (width 0.25) (layer B.Cu) (net 48))
+  (segment (start 206.85625 123) (end 206.25625 123) (width 0.25) (layer B.Cu) (net 49))
+  (segment (start 208.75625 121.1) (end 206.85625 123) (width 0.25) (layer B.Cu) (net 49))
+  (segment (start 204.94625 129.6525) (end 207.05625 131.7625) (width 0.25) (layer B.Cu) (net 49))
+  (segment (start 204.94625 124.46) (end 204.94625 129.6525) (width 0.25) (layer B.Cu) (net 49))
+  (segment (start 147.16125 66.3575) (end 149.70125 68.8975) (width 0.25) (layer B.Cu) (net 50))
+  (segment (start 134.46125 66.3575) (end 147.16125 66.3575) (width 0.25) (layer B.Cu) (net 50))
+  (zone (net 50) (net_name GND) (layer F.Cu) (hatch edge 0.508)
     (connect_pads (clearance 0.508))
     (min_thickness 0.254)
@@
     )
   )
-  (zone (net 49) (net_name GND) (layer B.Cu) (hatch edge 0.508)
+  (zone (net 50) (net_name GND) (layer B.Cu) (hatch edge 0.508)
     (connect_pads (clearance 0.508))
     (min_thickness 0.254)

Commit message: add uni name on the pcb
Other:
- board text added: "The Uni"

Commit message: add mounting holes to the uni pcb, also create a back plate folder in cases folder
Parts:
- added REF**: MountingHole_2.2mm_M2, MountingHole:MountingHole_2.2mm_M2, F.Cu at (256.4, 79.4)
- added REF**: MountingHole_2.2mm_M2, MountingHole:MountingHole_2.2mm_M2, F.Cu at (180.2, 79.4)
- added REF**: MountingHole_2.2mm_M2, MountingHole:MountingHole_2.2mm_M2, F.Cu at (199.2, 127.0)
- added REF**: MountingHole_2.2mm_M2, MountingHole:MountingHole_2.2mm_M2, F.Cu at (84.9, 127.0)
- added REF**: MountingHole_2.2mm_M2, MountingHole:MountingHole_2.2mm_M2, F.Cu at (104.0, 79.4)
- added REF**: MountingHole_2.2mm_M2, MountingHole:MountingHole_2.2mm_M2, F.Cu at (46.8, 79.4)
Routing:
- net col9: track 127.7 -> 133.4 mm
- net col10: track 146.4 -> 151.1 mm
- net col3: track 105.6 -> 103.0 mm
- net col4: track 88.3 -> 85.8 mm
- net col8: track 108.7 -> 110.2 mm
- net col6: track 113.2 -> 114.7 mm
- net col7: track 131.6 -> 133.1 mm
- net col2: track 123.9 -> 123.3 mm

Commit message: curvy trace and add reset
Parts:
- removed the REF** at (256.4, 79.4)
- removed the REF** at (180.2, 79.4)
- removed the REF** at (199.2, 127.0)
- removed the REF** at (84.9, 127.0)
- removed the REF** at (104.0, 79.4)
- removed the REF** at (46.8, 79.4)
- added REF**: m2, MountingHole:MountingHole_2.2mm_M2_DIN965_Pad, F.Cu at (84.9, 127.0)
- added REF**: m2, MountingHole:MountingHole_2.2mm_M2_DIN965_Pad, F.Cu at (104.0, 79.4)
- added REF**: m2, MountingHole:MountingHole_2.2mm_M2_DIN965_Pad, F.Cu at (180.2, 79.4)
- added REF**: m2, MountingHole:MountingHole_2.2mm_M2_DIN965_Pad, F.Cu at (256.4, 79.4)
- added REF**: m2, MountingHole:MountingHole_2.2mm_M2_DIN965_Pad, F.Cu at (46.8, 79.4)
- added REF**: m2, MountingHole:MountingHole_2.2mm_M2_DIN965_Pad, F.Cu at (199.2, 127.0)
- added SW1: SW_SPST, uni-footprints:jumper-reversible, F.Cu at (127.8, 63.5)
- moved U1 1.99 mm to (142.1, 79.8)
Connections:
- net Net-(U1-Pad21) renamed +5V
- U1 pad 1: Net-(U1-Pad1) -> unconnected-(U1-Pad1)
- U1 pad 2: Net-(U1-Pad2) -> unconnected-(U1-Pad2)
- U1 pad 22: Net-(U1-Pad22) -> reset
- U1 pad 24: Net-(U1-Pad24) -> unconnected-(U1-Pad24)
- U1 pad 5: Net-(U1-Pad5) -> unconnected-(U1-Pad5)
- U1 pad 6: Net-(U1-Pad6) -> unconnected-(U1-Pad6)
Routing:
- net col10: track 151.1 -> 168.3 mm
- net GND: track 16.3 -> 0.00 mm, vias 0 -> 15
- net reset: track 0.00 -> 11.8 mm
- net row1: track 241.0 -> 236.7 mm
- net row2: track 177.7 -> 182.0 mm
- net col0: track 122.8 -> 120.3 mm
- net col4: track 85.8 -> 83.6 mm
- net col1: track 101.9 -> 100.2 mm
- net col9: track 133.4 -> 132.1 mm
- net col2: track 123.3 -> 122.5 mm
- net col7: track 133.1 -> 132.4 mm
- net col6: track 114.7 -> 114.0 mm
- net row0: track 237.7 -> 237.1 mm
Other:
- net class Default removed
- board text added: "pro micro on top smooth side up"
- board text added: "stenokeyboards.com"
