File: unisplit_orthosteno.kicad_pcb (KiCad board)
At the start: 2 copper layers, 247.6 x 76.2 mm, 64 parts, among them SW1 SW_SPST, U1 ProMicro

Commit message: artwork
Parts:
- added G***: LOGO, uni-footprints:stenokeyboards-gregg, F.Cu at (142.1, 127.0)
- added G***: LOGO, uni-footprints:uni-gregg, B.Cu at (142.9, 119.1)
Other:
- board text removed: "Peter C. Park Design"

Commit message: fix fatal diode error
Connections:
- REF** pad 1: (no net) -> GND (x6)
Routing:
- net row2: track 182.0 -> 183.0 mm
- net GND: vias 15 -> 14
Changed lines of the file:
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@@
     (fp_circle (center 0 0) (end 1.9 0) (layer "Cmts.User") (width 0.15) (fill none))
     (fp_circle (center 0 0) (end 2.15 0) (layer "F.CrtYd") (width 0.05) (fill none))
-    (pad "1" thru_hole circle (at 0 0) (locked) (size 3.8 3.8) (drill 2.2) (layers *.Cu *.Mask))
+    (pad "1" thru_hole circle (at 0 0) (locked) (size 3.8 3.8) (drill 2.2) (layers *.Cu *.Mask)
+      (net 50 "GND"))
   )
   (footprint "MountingHole:MountingHole_2.2mm_M2_DIN965_Pad" (layer "F.Cu")
@@
     (fp_circle (center 0 0) (end 1.9 0) (layer "Cmts.User") (width 0.15) (fill none))
     (fp_circle (center 0 0) (end 2.15 0) (layer "F.CrtYd") (width 0.05) (fill none))
-    (pad "1" thru_hole circle (at 0 0) (locked) (size 3.8 3.8) (drill 2.2) (layers *.Cu *.Mask))
+    (pad "1" thru_hole circle (at 0 0) (locked) (size 3.8 3.8) (drill 2.2) (layers *.Cu *.Mask)
+      (net 50 "GND"))
   )
   (footprint "MountingHole:MountingHole_2.2mm_M2_DIN965_Pad" (layer "F.Cu")
@@
     (fp_circle (center 0 0) (end 1.9 0) (layer "Cmts.User") (width 0.15) (fill none))
     (fp_circle (center 0 0) (end 2.15 0) (layer "F.CrtYd") (width 0.05) (fill none))
-    (pad "1" thru_hole circle (at 0 0) (locked) (size 3.8 3.8) (drill 2.2) (layers *.Cu *.Mask))
+    (pad "1" thru_hole circle (at 0 0) (locked) (size 3.8 3.8) (drill 2.2) (layers *.Cu *.Mask)
+      (net 50 "GND"))
   )
   (footprint "MountingHole:MountingHole_2.2mm_M2_DIN965_Pad" (layer "F.Cu")
@@
     (fp_circle (center 0 0) (end 1.9 0) (layer "Cmts.User") (width 0.15) (fill none))
     (fp_circle (center 0 0) (end 2.15 0) (layer "F.CrtYd") (width 0.05) (fill none))
-    (pad "1" thru_hole circle (at 0 0) (locked) (size 3.8 3.8) (drill 2.2) (layers *.Cu *.Mask))
+    (pad "1" thru_hole circle (at 0 0) (locked) (size 3.8 3.8) (drill 2.2) (layers *.Cu *.Mask)
+      (net 50 "GND"))
   )
   (footprint "MountingHole:MountingHole_2.2mm_M2_DIN965_Pad" (layer "F.Cu")
@@
     (fp_circle (center 0 0) (end 1.9 0) (layer "Cmts.User") (width 0.15) (fill none))
     (fp_circle (center 0 0) (end 2.15 0) (layer "F.CrtYd") (width 0.05) (fill none))
-    (pad "1" thru_hole circle (at 0 0) (locked) (size 3.8 3.8) (drill 2.2) (layers *.Cu *.Mask))
+    (pad "1" thru_hole circle (at 0 0) (locked) (size 3.8 3.8) (drill 2.2) (layers *.Cu *.Mask)
+      (net 50 "GND"))
   )
   (footprint "uni-footprints:jumper-reversible" (layer "F.Cu")
@@
     (fp_circle (center 0 0) (end 1.9 0) (layer "Cmts.User") (width 0.15) (fill none))
     (fp_circle (center 0 0) (end 2.15 0) (layer "F.CrtYd") (width 0.05) (fill none))
-    (pad "1" thru_hole circle (at 0 0) (locked) (size 3.8 3.8) (drill 2.2) (layers *.Cu *.Mask))
+    (pad "1" thru_hole circle (at 0 0) (locked) (size 3.8 3.8) (drill 2.2) (layers *.Cu *.Mask)
+      (net 50 "GND"))
   )
   (footprint "Keebio-Parts:D_SOD123" (layer "B.Cu")
@@
     (effects (font (size 2 2) (thickness 0.2)) (justify mirror))
   )
-  (gr_text "The Uni" (at 141.732 119.0625) (layer "F.Mask")
+  (gr_text "The Uni" (at 141.732 119.85625) (layer "F.Mask")
     (effects (font (size 5 5) (thickness 0.3)))
   )
@@
   (arc (start 262.839143 86.067107) (mid 262.51472 86.28388) (end 262.132036 86.36) (width 0.25) (layer "B.Cu") (net 24))
   (arc (start 262.97493 92.43118) (mid 262.324611 91.45791) (end 262.09625 90.309859) (width 0.25) (layer "B.Cu") (net 24))
-  (segment (start 123.03125 124.100531) (end 123.03125 121.33858) (width 0.25) (layer "B.Cu") (net 25))
   (segment (start 171.804526 132.201724) (end 172.24375 131.7625) (width 0.25) (layer "B.Cu") (net 25))
   (segment (start 96.15625 131.7625) (end 96.595465 132.201715) (width 0.25) (layer "B.Cu") (net 25))
-  (segment (start 117.27003 131.502095) (end 117.792947 131.332189) (width 0.25) (layer "B.Cu") (net 25))
   (segment (start 95.717036 132.201714) (end 96.15625 131.7625) (width 0.25) (layer "B.Cu") (net 25))
-  (segment (start 116.735395 131.63045) (end 117.27003 131.502095) (width 0.25) (layer "B.Cu") (net 25))
+  (segment (start 120.122537 129.904614) (end 120.31898 129.71227) (width 0.25) (layer "B.Cu") (net 25))
   (segment (start 191.40625 131.7625) (end 191.845465 132.201715) (width 0.25) (layer "B.Cu") (net 25))
   (segment (start 117.059688 132.787511) (end 170.390312 132.787511) (width 0.25) (layer "B.Cu") (net 25))
   (segment (start 78.959678 132.787501) (end 94.302822 132.787501) (width 0.25) (layer "B.Cu") (net 25))
-  (segment (start 118.790821 130.872163) (end 119.259626 130.584879) (width 0.25) (layer "B.Cu") (net 25))
+  (segment (start 118.300921 131.121779) (end 118.790821 130.872163) (width 0.25) (layer "B.Cu") (net 25))
+  (segment (start 120.31898 129.71227) (end 120.981015 129.050235) (width 0.25) (layer "B.Cu") (net 25))
   (segment (start 172.24375 131.7625) (end 172.35625 131.7625) (width 0.25) (layer "B.Cu") (net 25))
   (segment (start 115.369291 131.7625) (end 115.644205 131.759601) (width 0.25) (layer "B.Cu") (net 25))
   (segment (start 134.029335 94.179439) (end 134.46125 93.74425) (width 0.25) (layer "B.Cu") (net 25))
-  (segment (start 119.259626 130.584879) (end 119.704445 130.261698) (width 0.25) (layer "B.Cu") (net 25))
-  (segment (start 117.792947 131.332189) (end 118.300921 131.121779) (width 0.25) (layer "B.Cu") (net 25))
   (segment (start 98.009678 132.787501) (end 113.352822 132.787501) (width 0.25) (layer "B.Cu") (net 25))
-  (segment (start 120.31898 129.71227) (end 120.981015 129.050235) (width 0.25) (layer "B.Cu") (net 25))
   (segment (start 210.017036 132.201714) (end 210.45625 131.7625) (width 0.25) (layer "B.Cu") (net 25))
+  (segment (start 123.03125 124.100531) (end 123.03125 121.33858) (width 0.25) (layer "B.Cu") (net 25))
   (segment (start 77.10625 131.7625) (end 77.545465 132.201715) (width 0.25) (layer "B.Cu") (net 25))
+  (segment (start 119.704445 130.261698) (end 120.122537 129.904614) (width 0.25) (layer "B.Cu") (net 25))
+  (segment (start 117.27003 131.502095) (end 117.792947 131.332189) (width 0.25) (layer "B.Cu") (net 25))
   (segment (start 172.35625 131.7625) (end 172.795465 132.201715) (width 0.25) (layer "B.Cu") (net 25))
-  (segment (start 120.122537 129.904614) (end 120.31898 129.71227) (width 0.25) (layer "B.Cu") (net 25))
+  (segment (start 116.735395 131.63045) (end 117.27003 131.502095) (width 0.25) (layer "B.Cu") (net 25))
+  (segment (start 118.790821 130.872163) (end 119.259626 130.584879) (width 0.25) (layer "B.Cu") (net 25))
   (segment (start 115.20625 131.7625) (end 115.369291 131.7625) (width 0.25) (layer "B.Cu") (net 25))
-  (segment (start 119.704445 130.261698) (end 120.122537 129.904614) (width 0.25) (layer "B.Cu") (net 25))
   (segment (start 190.967036 132.201714) (end 191.40625 131.7625) (width 0.25) (layer "B.Cu") (net 25))
   (segment (start 193.259678 132.787501) (end 208.602822 132.787501) (width 0.25) (layer "B.Cu") (net 25))
-  (segment (start 118.300921 131.121779) (end 118.790821 130.872163) (width 0.25) (layer "B.Cu") (net 25))
+  (segment (start 117.792947 131.332189) (end 118.300921 131.121779) (width 0.25) (layer "B.Cu") (net 25))
   (segment (start 174.209678 132.787501) (end 189.552822 132.787501) (width 0.25) (layer "B.Cu") (net 25))
   (segment (start 114.767036 132.201714) (end 115.20625 131.7625) (width 0.25) (layer "B.Cu") (net 25))
+  (segment (start 119.259626 130.584879) (end 119.704445 130.261698) (width 0.25) (layer "B.Cu") (net 25))
+  (segment (start 115.20625 131.7625) (end 116.735395 131.63045) (width 0.25) (layer "B.Cu") (net 25))
   (segment (start 115.20625 131.7625) (end 115.645475 132.201725) (width 0.25) (layer "B.Cu") (net 25))
-  (segment (start 116.192337 131.716462) (end 116.735395 131.63045) (width 0.25) (layer "B.Cu") (net 25))
   (arc (start 117.059688 132.787511) (mid 116.294321 132.63527) (end 115.645475 132.201725) (width 0.25) (layer "B.Cu") (net 25))
   (arc (start 189.552822 132.787501) (mid 190.318189 132.63526) (end 190.967036 132.201714) (width 0.25) (layer "B.Cu") (net 25))
   (arc (start 170.390312 132.787511) (mid 171.155679 132.63527) (end 171.804526 132.201724) (width 0.25) (layer "B.Cu") (net 25))
   (arc (start 191.845465 132.201715) (mid 192.494311 132.63526) (end 193.259678 132.787501) (width 0.25) (layer "B.Cu") (net 25))
+  (arc (start 120.981015 129.050235) (mid 122.498411 126.779292) (end 123.03125 124.100531) (width 0.25) (layer "B.Cu") (net 25))
   (arc (start 172.795465 132.201715) (mid 173.444311 132.63526) (end 174.209678 132.787501) (width 0.25) (layer "B.Cu") (net 25))
   (arc (start 123.03125 121.33858) (mid 126.001786 106.404687) (end 134.461157 93.744343) (width 0.25) (layer "B.Cu") (net 25))
-  (arc (start 120.981015 129.050235) (mid 122.498411 126.779292) (end 123.03125 124.100531) (width 0.25) (layer "B.Cu") (net 25))
   (arc (start 77.545465 132.201715) (mid 78.194311 132.63526) (end 78.959678 132.787501) (width 0.25) (layer "B.Cu") (net 25))
   (arc (start 210.017036 132.201714) (mid 209.368189 132.63526) (end 208.602822 132.787501) (width 0.25) (layer "B.Cu") (net 25))
@@
   (via (at 208.788 85.344) (size 0.8) (drill 0.4) (layers "F.Cu" "B.Cu") (free) (net 50))
   (via (at 165.354 91.059) (size 0.8) (drill 0.4) (layers "F.Cu" "B.Cu") (free) (net 50))
-  (via (at 176.657 78.105) (size 0.8) (drill 0.4) (layers "F.Cu" "B.Cu") (free) (net 50))
   (via (at 56.388 85.344) (size 0.8) (drill 0.4) (layers "F.Cu" "B.Cu") (free) (net 50))
   (via (at 170.688 85.344) (size 0.8) (drill 0.4) (layers "F.Cu" "B.Cu") (free) (net 50))

Commit message: add tooling and order number
Parts:
- added jlc**: jlc-tooling-hole, uni-footprints:jlc-tooling-hole, F.Cu at (215.9, 134.1)
- added jlc**: jlc-tooling-hole, uni-footprints:jlc-tooling-hole, F.Cu at (29.4, 61.9)
Other:
- board text added: "JLCJLCJLCJLC"
Changed lines of the file:
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@@
       (net 50 "GND"))
+  )
+  (footprint "uni-footprints:jlc-tooling-hole" (layer "F.Cu")
+    (at 215.9 134.14375)
+    (fp_text reference "jlc**" (at 0 -0.5 unlocked) (layer "F.Fab")
+      (effects (font (size 1 1) (thickness 0.15)))
+    )
+    (fp_text value "jlc-tooling-hole" (at 0 1 unlocked) (layer "F.Fab")
+      (effects (font (size 1 1) (thickness 0.15)))
+    )
+    (pad "" np_thru_hole circle (at 0 0) (locked) (size 1.152 1.152) (drill 1.152) (layers F&B.Cu *.Mask)
+      (solder_mask_margin 0.148) (solder_paste_margin 1.152) (zone_connect 0))
   )
   (footprint "MountingHole:MountingHole_2.2mm_M2_DIN965_Pad" (layer "F.Cu")
@@
     (pad "1" thru_hole circle (at 0 0) (locked) (size 3.8 3.8) (drill 2.2) (layers *.Cu *.Mask)
       (net 50 "GND"))
+  )
+  (footprint "uni-footprints:jlc-tooling-hole" (layer "F.Cu")
+    (at 29.36875 61.9125)
+    (fp_text reference "jlc**" (at 0 -0.5 unlocked) (layer "F.Fab")
+      (effects (font (size 1 1) (thickness 0.15)))
+    )
+    (fp_text value "jlc-tooling-hole" (at 0 1 unlocked) (layer "F.Fab")
+      (effects (font (size 1 1) (thickness 0.15)))
+    )
+    (pad "" np_thru_hole circle (at 0 0) (locked) (size 1.152 1.152) (drill 1.152) (layers F&B.Cu *.Mask)
+      (solder_mask_margin 0.148) (solder_paste_margin 1.152) (zone_connect 0))
   )
   (footprint "uni-footprints:jumper-reversible" (layer "F.Cu")
@@
   (gr_arc (start 220.6625 100.80625) (end 220.6625 98.425) (angle -90) (layer "Edge.Cuts") (width 0.05))
   (gr_arc (start 215.9 134.14375) (end 215.9 136.525) (angle -90) (layer "Edge.Cuts") (width 0.05))
+  (gr_text "JLCJLCJLCJLC" (at 141.2875 134.9375) (layer "B.SilkS")
+    (effects (font (size 0.8 0.8) (thickness 0.1)) (justify mirror))
+  )
   (gr_text "pro micro on top\nsmooth side up" (at 142.08125 79.375 90) (layer "F.SilkS")
     (effects (font (size 1 1) (thickness 0.25)))
