File: unisplit_orthosteno.kicad_pcb (KiCad board)
At the start: 2 copper layers, 247.6 x 76.2 mm, 68 parts, among them SW1 SW_SPST, U1 ProMicro

Commit message: add more mounting holes
Parts:
- added REF**: m2, MountingHole:MountingHole_2.2mm_M2_DIN965_Pad, F.Cu at (120.7, 62.7)
- added REF**: m2, MountingHole:MountingHole_2.2mm_M2_DIN965_Pad, F.Cu at (30.2, 96.0)
- added REF**: m2, MountingHole:MountingHole_2.2mm_M2_DIN965_Pad, F.Cu at (217.5, 97.6)
- added REF**: m2, MountingHole:MountingHole_2.2mm_M2_DIN965_Pad, F.Cu at (66.7, 97.6)
- added REF**: m2, MountingHole:MountingHole_2.2mm_M2_DIN965_Pad, F.Cu at (273.1, 62.7)
- added REF**: m2, MountingHole:MountingHole_2.2mm_M2_DIN965_Pad, F.Cu at (68.3, 134.1)
- added REF**: m2, MountingHole:MountingHole_2.2mm_M2_DIN965_Pad, F.Cu at (273.1, 96.0)
- added REF**: m2, MountingHole:MountingHole_2.2mm_M2_DIN965_Pad, F.Cu at (215.9, 134.1)
- added REF**: m2, MountingHole:MountingHole_2.2mm_M2_DIN965_Pad, F.Cu at (163.5, 62.7)
- added REF**: m2, MountingHole:MountingHole_2.2mm_M2_DIN965_Pad, F.Cu at (30.2, 62.7)
- moved jlc** 17.5 mm to (46.8, 62.7)
- moved jlc** 3.37 mm to (213.5, 131.8)
Changed lines of the file:
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@@
       (net 49 "Net-(D28-Pad2)") (pinfunction "ROW") (pintype "passive"))
+  )
+  (footprint "MountingHole:MountingHole_2.2mm_M2_DIN965_Pad" (layer "F.Cu")
+    (at 120.65 62.70625)
+    (descr "Mounting Hole 2.2mm, M2, DIN965")
+    (tags "mounting hole 2.2mm m2 din965")
+    (attr exclude_from_pos_files exclude_from_bom)
+    (fp_text reference "REF**" (at 0 -2.9) (layer "F.SilkS") hide
+      (effects (font (size 1 1) (thickness 0.15)))
+    )
+    (fp_text value "m2" (at 0 2.9) (layer "F.Fab")
+      (effects (font (size 1 1) (thickness 0.15)))
+    )
+    (fp_text user "${REFERENCE}" (at 0.3 0) (layer "F.Fab")
+      (effects (font (size 1 1) (thickness 0.15)))
+    )
+    (fp_circle (center 0 0) (end 1.9 0) (layer "Cmts.User") (width 0.15) (fill none))
+    (fp_circle (center 0 0) (end 2.15 0) (layer "F.CrtYd") (width 0.05) (fill none))
+    (pad "1" thru_hole circle (at 0 0) (locked) (size 3.8 3.8) (drill 2.2) (layers *.Cu *.Mask)
+      (net 50 "GND"))
   )
   (footprint "uni-footprints:stenokeyboards-gregg" (layer "F.Cu")
@@
   )
   (footprint "MountingHole:MountingHole_2.2mm_M2_DIN965_Pad" (layer "F.Cu")
+    (at 273.05 96.04375)
+    (descr "Mounting Hole 2.2mm, M2, DIN965")
+    (tags "mounting hole 2.2mm m2 din965")
+    (attr exclude_from_pos_files exclude_from_bom)
+    (fp_text reference "REF**" (at 0 -2.9) (layer "F.SilkS") hide
+      (effects (font (size 1 1) (thickness 0.15)))
+    )
+    (fp_text value "m2" (at 0 2.9) (layer "F.Fab")
+      (effects (font (size 1 1) (thickness 0.15)))
+    )
+    (fp_text user "${REFERENCE}" (at 0.3 0) (layer "F.Fab")
+      (effects (font (size 1 1) (thickness 0.15)))
+    )
+    (fp_circle (center 0 0) (end 1.9 0) (layer "Cmts.User") (width 0.15) (fill none))
+    (fp_circle (center 0 0) (end 2.15 0) (layer "F.CrtYd") (width 0.05) (fill none))
+    (pad "1" thru_hole circle (at 0 0) (locked) (size 3.8 3.8) (drill 2.2) (layers *.Cu *.Mask)
+      (net 50 "GND"))
+  )
+  (footprint "MountingHole:MountingHole_2.2mm_M2_DIN965_Pad" (layer "F.Cu")
+    (at 215.9 134.14375)
+    (descr "Mounting Hole 2.2mm, M2, DIN965")
+    (tags "mounting hole 2.2mm m2 din965")
+    (attr exclude_from_pos_files exclude_from_bom)
+    (fp_text reference "REF**" (at 0 -2.9) (layer "F.SilkS") hide
+      (effects (font (size 1 1) (thickness 0.15)))
+    )
+    (fp_text value "m2" (at 0 2.9) (layer "F.Fab")
+      (effects (font (size 1 1) (thickness 0.15)))
+    )
+    (fp_text user "${REFERENCE}" (at 0.3 0) (layer "F.Fab")
+      (effects (font (size 1 1) (thickness 0.15)))
+    )
+    (fp_circle (center 0 0) (end 1.9 0) (layer "Cmts.User") (width 0.15) (fill none))
+    (fp_circle (center 0 0) (end 2.15 0) (layer "F.CrtYd") (width 0.05) (fill none))
+    (pad "1" thru_hole circle (at 0 0) (locked) (size 3.8 3.8) (drill 2.2) (layers *.Cu *.Mask)
+      (net 50 "GND"))
+  )
+  (footprint "MountingHole:MountingHole_2.2mm_M2_DIN965_Pad" (layer "F.Cu")
     (at 103.98125 79.375)
     (descr "Mounting Hole 2.2mm, M2, DIN965")
@@
       (net 50 "GND"))
   )
+  (footprint "MountingHole:MountingHole_2.2mm_M2_DIN965_Pad" (layer "F.Cu")
+    (at 163.5125 62.70625)
+    (descr "Mounting Hole 2.2mm, M2, DIN965")
+    (tags "mounting hole 2.2mm m2 din965")
+    (attr exclude_from_pos_files exclude_from_bom)
+    (fp_text reference "REF**" (at 0 -2.9) (layer "F.SilkS") hide
+      (effects (font (size 1 1) (thickness 0.15)))
+    )
+    (fp_text value "m2" (at 0 2.9) (layer "F.Fab")
+      (effects (font (size 1 1) (thickness 0.15)))
+    )
+    (fp_text user "${REFERENCE}" (at 0.3 0) (layer "F.Fab")
+      (effects (font (size 1 1) (thickness 0.15)))
+    )
+    (fp_circle (center 0 0) (end 1.9 0) (layer "Cmts.User") (width 0.15) (fill none))
+    (fp_circle (center 0 0) (end 2.15 0) (layer "F.CrtYd") (width 0.05) (fill none))
+    (pad "1" thru_hole circle (at 0 0) (locked) (size 3.8 3.8) (drill 2.2) (layers *.Cu *.Mask)
+      (net 50 "GND"))
+  )
+  (footprint "MountingHole:MountingHole_2.2mm_M2_DIN965_Pad" (layer "F.Cu")
+    (at 30.1625 62.70625)
+    (descr "Mounting Hole 2.2mm, M2, DIN965")
+    (tags "mounting hole 2.2mm m2 din965")
+    (attr exclude_from_pos_files exclude_from_bom)
+    (fp_text reference "REF**" (at 0 -2.9) (layer "F.SilkS") hide
+      (effects (font (size 1 1) (thickness 0.15)))
+    )
+    (fp_text value "m2" (at 0 2.9) (layer "F.Fab")
+      (effects (font (size 1 1) (thickness 0.15)))
+    )
+    (fp_text user "${REFERENCE}" (at 0.3 0) (layer "F.Fab")
+      (effects (font (size 1 1) (thickness 0.15)))
+    )
+    (fp_circle (center 0 0) (end 1.9 0) (layer "Cmts.User") (width 0.15) (fill none))
+    (fp_circle (center 0 0) (end 2.15 0) (layer "F.CrtYd") (width 0.05) (fill none))
+    (pad "1" thru_hole circle (at 0 0) (locked) (size 3.8 3.8) (drill 2.2) (layers *.Cu *.Mask)
+      (net 50 "GND"))
+  )
   (footprint "uni-footprints:jlc-tooling-hole" (layer "F.Cu")
-    (at 215.9 134.14375)
+    (at 213.51875 131.7625)
     (fp_text reference "jlc**" (at 0 -0.5 unlocked) (layer "F.Fab")
       (effects (font (size 1 1) (thickness 0.15)))
@@
   )
   (footprint "uni-footprints:jlc-tooling-hole" (layer "F.Cu")
-    (at 29.36875 61.9125)
+    (at 46.83125 62.70625)
     (fp_text reference "jlc**" (at 0 -0.5 unlocked) (layer "F.Fab")
       (effects (font (size 1 1) (thickness 0.15)))
@@
       (solder_mask_margin 0.148) (solder_paste_margin 1.152) (zone_connect 0))
   )
+  (footprint "MountingHole:MountingHole_2.2mm_M2_DIN965_Pad" (layer "F.Cu")
+    (at 30.1625 96.04375)
+    (descr "Mounting Hole 2.2mm, M2, DIN965")
+    (tags "mounting hole 2.2mm m2 din965")
+    (attr exclude_from_pos_files exclude_from_bom)
+    (fp_text reference "REF**" (at 0 -2.9) (layer "F.SilkS") hide
+      (effects (font (size 1 1) (thickness 0.15)))
+    )
+    (fp_text value "m2" (at 0 2.9) (layer "F.Fab")
+      (effects (font (size 1 1) (thickness 0.15)))
+    )
+    (fp_text user "${REFERENCE}" (at 0.3 0) (layer "F.Fab")
+      (effects (font (size 1 1) (thickness 0.15)))
+    )
+    (fp_circle (center 0 0) (end 1.9 0) (layer "Cmts.User") (width 0.15) (fill none))
+    (fp_circle (center 0 0) (end 2.15 0) (layer "F.CrtYd") (width 0.05) (fill none))
+    (pad "1" thru_hole circle (at 0 0) (locked) (size 3.8 3.8) (drill 2.2) (layers *.Cu *.Mask)
+      (net 50 "GND"))
+  )
+  (footprint "MountingHole:MountingHole_2.2mm_M2_DIN965_Pad" (layer "F.Cu")
+    (at 217.4875 97.63125)
+    (descr "Mounting Hole 2.2mm, M2, DIN965")
+    (tags "mounting hole 2.2mm m2 din965")
+    (attr exclude_from_pos_files exclude_from_bom)
+    (fp_text reference "REF**" (at 0 -2.9) (layer "F.SilkS") hide
+      (effects (font (size 1 1) (thickness 0.15)))
+    )
+    (fp_text value "m2" (at 0 2.9) (layer "F.Fab")
+      (effects (font (size 1 1) (thickness 0.15)))
+    )
+    (fp_text user "${REFERENCE}" (at 0.3 0) (layer "F.Fab")
+      (effects (font (size 1 1) (thickness 0.15)))
+    )
+    (fp_circle (center 0 0) (end 1.9 0) (layer "Cmts.User") (width 0.15) (fill none))
+    (fp_circle (center 0 0) (end 2.15 0) (layer "F.CrtYd") (width 0.05) (fill none))
+    (pad "1" thru_hole circle (at 0 0) (locked) (size 3.8 3.8) (drill 2.2) (layers *.Cu *.Mask)
+      (net 50 "GND"))
+  )
+  (footprint "MountingHole:MountingHole_2.2mm_M2_DIN965_Pad" (layer "F.Cu")
+    (at 66.675 97.63125)
+    (descr "Mounting Hole 2.2mm, M2, DIN965")
+    (tags "mounting hole 2.2mm m2 din965")
+    (attr exclude_from_pos_files exclude_from_bom)
+    (fp_text reference "REF**" (at 0 -2.9) (layer "F.SilkS") hide
+      (effects (font (size 1 1) (thickness 0.15)))
+    )
+    (fp_text value "m2" (at 0 2.9) (layer "F.Fab")
+      (effects (font (size 1 1) (thickness 0.15)))
+    )
+    (fp_text user "${REFERENCE}" (at 0.3 0) (layer "F.Fab")
+      (effects (font (size 1 1) (thickness 0.15)))
+    )
+    (fp_circle (center 0 0) (end 1.9 0) (layer "Cmts.User") (width 0.15) (fill none))
+    (fp_circle (center 0 0) (end 2.15 0) (layer "F.CrtYd") (width 0.05) (fill none))
+    (pad "1" thru_hole circle (at 0 0) (locked) (size 3.8 3.8) (drill 2.2) (layers *.Cu *.Mask)
+      (net 50 "GND"))
+  )
+  (footprint "MountingHole:MountingHole_2.2mm_M2_DIN965_Pad" (layer "F.Cu")
+    (at 273.05 62.70625)
+    (descr "Mounting Hole 2.2mm, M2, DIN965")
+    (tags "mounting hole 2.2mm m2 din965")
+    (attr exclude_from_pos_files exclude_from_bom)
+    (fp_text reference "REF**" (at 0 -2.9) (layer "F.SilkS") hide
+      (effects (font (size 1 1) (thickness 0.15)))
+    )
+    (fp_text value "m2" (at 0 2.9) (layer "F.Fab")
+      (effects (font (size 1 1) (thickness 0.15)))
+    )
+    (fp_text user "${REFERENCE}" (at 0.3 0) (layer "F.Fab")
+      (effects (font (size 1 1) (thickness 0.15)))
+    )
+    (fp_circle (center 0 0) (end 1.9 0) (layer "Cmts.User") (width 0.15) (fill none))
+    (fp_circle (center 0 0) (end 2.15 0) (layer "F.CrtYd") (width 0.05) (fill none))
+    (pad "1" thru_hole circle (at 0 0) (locked) (size 3.8 3.8) (drill 2.2) (layers *.Cu *.Mask)
+      (net 50 "GND"))
+  )
+  (footprint "MountingHole:MountingHole_2.2mm_M2_DIN965_Pad" (layer "F.Cu")
+    (at 68.2625 134.14375)
+    (descr "Mounting Hole 2.2mm, M2, DIN965")
+    (tags "mounting hole 2.2mm m2 din965")
+    (attr exclude_from_pos_files exclude_from_bom)
+    (fp_text reference "REF**" (at 0 -2.9) (layer "F.SilkS") hide
+      (effects (font (size 1 1) (thickness 0.15)))
+    )
+    (fp_text value "m2" (at 0 2.9) (layer "F.Fab")
+      (effects (font (size 1 1) (thickness 0.15)))
+    )
+    (fp_text user "${REFERENCE}" (at 0.3 0) (layer "F.Fab")
+      (effects (font (size 1 1) (thickness 0.15)))
+    )
+    (fp_circle (center 0 0) (end 1.9 0) (layer "Cmts.User") (width 0.15) (fill none))
+    (fp_circle (center 0 0) (end 2.15 0) (layer "F.CrtYd") (width 0.05) (fill none))
+    (pad "1" thru_hole circle (at 0 0) (locked) (size 3.8 3.8) (drill 2.2) (layers *.Cu *.Mask)
+      (net 50 "GND"))
+  )
   (footprint "uni-footprints:jumper-reversible" (layer "F.Cu")

Commit message: get rid of extra nuisance mounting holes
Parts:
- removed the REF** at (30.2, 96.0)
- removed the REF** at (217.5, 97.6)
- removed the REF** at (66.7, 97.6)
- removed the REF** at (273.1, 62.7)
- removed the REF** at (68.3, 134.1)
- removed the REF** at (273.1, 96.0)
- removed the REF** at (215.9, 134.1)
- removed the REF** at (30.2, 62.7)
Changed lines of the file:
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@@
-  )
-  (footprint "MountingHole:MountingHole_2.2mm_M2_DIN965_Pad" (layer "F.Cu")
-    (at 273.05 96.04375)
-    (descr "Mounting Hole 2.2mm, M2, DIN965")
-    (tags "mounting hole 2.2mm m2 din965")
-    (attr exclude_from_pos_files exclude_from_bom)
-    (fp_text reference "REF**" (at 0 -2.9) (layer "F.SilkS") hide
-      (effects (font (size 1 1) (thickness 0.15)))
-    )
-    (fp_text value "m2" (at 0 2.9) (layer "F.Fab")
-      (effects (font (size 1 1) (thickness 0.15)))
-    )
-    (fp_text user "${REFERENCE}" (at 0.3 0) (layer "F.Fab")
-      (effects (font (size 1 1) (thickness 0.15)))
-    )
-    (fp_circle (center 0 0) (end 1.9 0) (layer "Cmts.User") (width 0.15) (fill none))
-    (fp_circle (center 0 0) (end 2.15 0) (layer "F.CrtYd") (width 0.05) (fill none))
-    (pad "1" thru_hole circle (at 0 0) (locked) (size 3.8 3.8) (drill 2.2) (layers *.Cu *.Mask)
-      (net 50 "GND"))
-  )
-  (footprint "MountingHole:MountingHole_2.2mm_M2_DIN965_Pad" (layer "F.Cu")
-    (at 215.9 134.14375)
-    (descr "Mounting Hole 2.2mm, M2, DIN965")
-    (tags "mounting hole 2.2mm m2 din965")
-    (attr exclude_from_pos_files exclude_from_bom)
-    (fp_text reference "REF**" (at 0 -2.9) (layer "F.SilkS") hide
-      (effects (font (size 1 1) (thickness 0.15)))
-    )
-    (fp_text value "m2" (at 0 2.9) (layer "F.Fab")
-      (effects (font (size 1 1) (thickness 0.15)))
-    )
-    (fp_text user "${REFERENCE}" (at 0.3 0) (layer "F.Fab")
-      (effects (font (size 1 1) (thickness 0.15)))
-    )
-    (fp_circle (center 0 0) (end 1.9 0) (layer "Cmts.User") (width 0.15) (fill none))
-    (fp_circle (center 0 0) (end 2.15 0) (layer "F.CrtYd") (width 0.05) (fill none))
-    (pad "1" thru_hole circle (at 0 0) (locked) (size 3.8 3.8) (drill 2.2) (layers *.Cu *.Mask)
-      (net 50 "GND"))
   )
   (footprint "MountingHole:MountingHole_2.2mm_M2_DIN965_Pad" (layer "F.Cu")
@@
   (footprint "MountingHole:MountingHole_2.2mm_M2_DIN965_Pad" (layer "F.Cu")
     (at 163.5125 62.70625)
-    (descr "Mounting Hole 2.2mm, M2, DIN965")
-    (tags "mounting hole 2.2mm m2 din965")
-    (attr exclude_from_pos_files exclude_from_bom)
-    (fp_text reference "REF**" (at 0 -2.9) (layer "F.SilkS") hide
-      (effects (font (size 1 1) (thickness 0.15)))
-    )
-    (fp_text value "m2" (at 0 2.9) (layer "F.Fab")
-      (effects (font (size 1 1) (thickness 0.15)))
-    )
-    (fp_text user "${REFERENCE}" (at 0.3 0) (layer "F.Fab")
-      (effects (font (size 1 1) (thickness 0.15)))
-    )
-    (fp_circle (center 0 0) (end 1.9 0) (layer "Cmts.User") (width 0.15) (fill none))
-    (fp_circle (center 0 0) (end 2.15 0) (layer "F.CrtYd") (width 0.05) (fill none))
-    (pad "1" thru_hole circle (at 0 0) (locked) (size 3.8 3.8) (drill 2.2) (layers *.Cu *.Mask)
-      (net 50 "GND"))
-  )
-  (footprint "MountingHole:MountingHole_2.2mm_M2_DIN965_Pad" (layer "F.Cu")
-    (at 30.1625 62.70625)
     (descr "Mounting Hole 2.2mm, M2, DIN965")
     (tags "mounting hole 2.2mm m2 din965")
@@
       (solder_mask_margin 0.148) (solder_paste_margin 1.152) (zone_connect 0))
   )
-  (footprint "MountingHole:MountingHole_2.2mm_M2_DIN965_Pad" (layer "F.Cu")
-    (at 30.1625 96.04375)
-    (descr "Mounting Hole 2.2mm, M2, DIN965")
-    (tags "mounting hole 2.2mm m2 din965")
-    (attr exclude_from_pos_files exclude_from_bom)
-    (fp_text reference "REF**" (at 0 -2.9) (layer "F.SilkS") hide
-      (effects (font (size 1 1) (thickness 0.15)))
-    )
-    (fp_text value "m2" (at 0 2.9) (layer "F.Fab")
-      (effects (font (size 1 1) (thickness 0.15)))
-    )
-    (fp_text user "${REFERENCE}" (at 0.3 0) (layer "F.Fab")
-      (effects (font (size 1 1) (thickness 0.15)))
-    )
-    (fp_circle (center 0 0) (end 1.9 0) (layer "Cmts.User") (width 0.15) (fill none))
-    (fp_circle (center 0 0) (end 2.15 0) (layer "F.CrtYd") (width 0.05) (fill none))
-    (pad "1" thru_hole circle (at 0 0) (locked) (size 3.8 3.8) (drill 2.2) (layers *.Cu *.Mask)
-      (net 50 "GND"))
-  )
-  (footprint "MountingHole:MountingHole_2.2mm_M2_DIN965_Pad" (layer "F.Cu")
-    (at 217.4875 97.63125)
-    (descr "Mounting Hole 2.2mm, M2, DIN965")
-    (tags "mounting hole 2.2mm m2 din965")
-    (attr exclude_from_pos_files exclude_from_bom)
-    (fp_text reference "REF**" (at 0 -2.9) (layer "F.SilkS") hide
-      (effects (font (size 1 1) (thickness 0.15)))
-    )
-    (fp_text value "m2" (at 0 2.9) (layer "F.Fab")
-      (effects (font (size 1 1) (thickness 0.15)))
-    )
-    (fp_text user "${REFERENCE}" (at 0.3 0) (layer "F.Fab")
-      (effects (font (size 1 1) (thickness 0.15)))
-    )
-    (fp_circle (center 0 0) (end 1.9 0) (layer "Cmts.User") (width 0.15) (fill none))
-    (fp_circle (center 0 0) (end 2.15 0) (layer "F.CrtYd") (width 0.05) (fill none))
-    (pad "1" thru_hole circle (at 0 0) (locked) (size 3.8 3.8) (drill 2.2) (layers *.Cu *.Mask)
-      (net 50 "GND"))
-  )
-  (footprint "MountingHole:MountingHole_2.2mm_M2_DIN965_Pad" (layer "F.Cu")
-    (at 66.675 97.63125)
-    (descr "Mounting Hole 2.2mm, M2, DIN965")
-    (tags "mounting hole 2.2mm m2 din965")
-    (attr exclude_from_pos_files exclude_from_bom)
-    (fp_text reference "REF**" (at 0 -2.9) (layer "F.SilkS") hide
-      (effects (font (size 1 1) (thickness 0.15)))
-    )
-    (fp_text value "m2" (at 0 2.9) (layer "F.Fab")
-      (effects (font (size 1 1) (thickness 0.15)))
-    )
-    (fp_text user "${REFERENCE}" (at 0.3 0) (layer "F.Fab")
-      (effects (font (size 1 1) (thickness 0.15)))
-    )
-    (fp_circle (center 0 0) (end 1.9 0) (layer "Cmts.User") (width 0.15) (fill none))
-    (fp_circle (center 0 0) (end 2.15 0) (layer "F.CrtYd") (width 0.05) (fill none))
-    (pad "1" thru_hole circle (at 0 0) (locked) (size 3.8 3.8) (drill 2.2) (layers *.Cu *.Mask)
-      (net 50 "GND"))
-  )
-  (footprint "MountingHole:MountingHole_2.2mm_M2_DIN965_Pad" (layer "F.Cu")
-    (at 273.05 62.70625)
-    (descr "Mounting Hole 2.2mm, M2, DIN965")
-    (tags "mounting hole 2.2mm m2 din965")
-    (attr exclude_from_pos_files exclude_from_bom)
-    (fp_text reference "REF**" (at 0 -2.9) (layer "F.SilkS") hide
-      (effects (font (size 1 1) (thickness 0.15)))
-    )
-    (fp_text value "m2" (at 0 2.9) (layer "F.Fab")
-      (effects (font (size 1 1) (thickness 0.15)))
-    )
-    (fp_text user "${REFERENCE}" (at 0.3 0) (layer "F.Fab")
-      (effects (font (size 1 1) (thickness 0.15)))
-    )
-    (fp_circle (center 0 0) (end 1.9 0) (layer "Cmts.User") (width 0.15) (fill none))
-    (fp_circle (center 0 0) (end 2.15 0) (layer "F.CrtYd") (width 0.05) (fill none))
-    (pad "1" thru_hole circle (at 0 0) (locked) (size 3.8 3.8) (drill 2.2) (layers *.Cu *.Mask)
-      (net 50 "GND"))
-  )
-  (footprint "MountingHole:MountingHole_2.2mm_M2_DIN965_Pad" (layer "F.Cu")
-    (at 68.2625 134.14375)
-    (descr "Mounting Hole 2.2mm, M2, DIN965")
-    (tags "mounting hole 2.2mm m2 din965")
-    (attr exclude_from_pos_files exclude_from_bom)
-    (fp_text reference "REF**" (at 0 -2.9) (layer "F.SilkS") hide
-      (effects (font (size 1 1) (thickness 0.15)))
-    )
-    (fp_text value "m2" (at 0 2.9) (layer "F.Fab")
-      (effects (font (size 1 1) (thickness 0.15)))
-    )
-    (fp_text user "${REFERENCE}" (at 0.3 0) (layer "F.Fab")
-      (effects (font (size 1 1) (thickness 0.15)))
-    )
-    (fp_circle (center 0 0) (end 1.9 0) (layer "Cmts.User") (width 0.15) (fill none))
-    (fp_circle (center 0 0) (end 2.15 0) (layer "F.CrtYd") (width 0.05) (fill none))
-    (pad "1" thru_hole circle (at 0 0) (locked) (size 3.8 3.8) (drill 2.2) (layers *.Cu *.Mask)
-      (net 50 "GND"))
-  )
   (footprint "uni-footprints:jumper-reversible" (layer "F.Cu")

Commit message: update gerbers.
Parts:
- removed the REF** at (120.7, 62.7)
- removed the REF** at (163.5, 62.7)
Changed lines of the file:
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@@
       (drillshape 0)
       (scaleselection 1)
-      (outputdirectory "Gerbers/v2.1/")
+      (outputdirectory "Gerbers/v2/")
     )
   )
@@
     (pad "2" thru_hole oval (at -3.81 -2.54 48.1) (locked) (size 4.211556 2.25) (drill 1.47 (offset 0.980778 0)) (layers *.Cu *.Mask)
       (net 49 "Net-(D28-Pad2)") (pinfunction "ROW") (pintype "passive"))
-  )
-  (footprint "MountingHole:MountingHole_2.2mm_M2_DIN965_Pad" (layer "F.Cu")
-    (at 120.65 62.70625)
-    (descr "Mounting Hole 2.2mm, M2, DIN965")
-    (tags "mounting hole 2.2mm m2 din965")
-    (attr exclude_from_pos_files exclude_from_bom)
-    (fp_text reference "REF**" (at 0 -2.9) (layer "F.SilkS") hide
-      (effects (font (size 1 1) (thickness 0.15)))
-    )
-    (fp_text value "m2" (at 0 2.9) (layer "F.Fab")
-      (effects (font (size 1 1) (thickness 0.15)))
-    )
-    (fp_text user "${REFERENCE}" (at 0.3 0) (layer "F.Fab")
-      (effects (font (size 1 1) (thickness 0.15)))
-    )
-    (fp_circle (center 0 0) (end 1.9 0) (layer "Cmts.User") (width 0.15) (fill none))
-    (fp_circle (center 0 0) (end 2.15 0) (layer "F.CrtYd") (width 0.05) (fill none))
-    (pad "1" thru_hole circle (at 0 0) (locked) (size 3.8 3.8) (drill 2.2) (layers *.Cu *.Mask)
-      (net 50 "GND"))
   )
   (footprint "uni-footprints:stenokeyboards-gregg" (layer "F.Cu")
@@
     (descr "Mounting Hole 2.2mm, M2, DIN965")
     (tags "mounting hole 2.2mm m2 din965")
-    (attr exclude_from_pos_files exclude_from_bom)
-    (fp_text reference "REF**" (at 0 -2.9) (layer "F.SilkS") hide
-      (effects (font (size 1 1) (thickness 0.15)))
-    )
-    (fp_text value "m2" (at 0 2.9) (layer "F.Fab")
-      (effects (font (size 1 1) (thickness 0.15)))
-    )
-    (fp_text user "${REFERENCE}" (at 0.3 0) (layer "F.Fab")
-      (effects (font (size 1 1) (thickness 0.15)))
-    )
-    (fp_circle (center 0 0) (end 1.9 0) (layer "Cmts.User") (width 0.15) (fill none))
-    (fp_circle (center 0 0) (end 2.15 0) (layer "F.CrtYd") (width 0.05) (fill none))
-    (pad "1" thru_hole circle (at 0 0) (locked) (size 3.8 3.8) (drill 2.2) (layers *.Cu *.Mask)
-      (net 50 "GND"))
-  )
-  (footprint "MountingHole:MountingHole_2.2mm_M2_DIN965_Pad" (layer "F.Cu")
-    (at 163.5125 62.70625)
-    (descr "Mounting Hole 2.2mm, M2, DIN965")
-    (tags "mounting hole 2.2mm m2 din965")

Commit message: docs
Parts:
- moved jlc** 16.7 mm to (30.2, 62.7)
- moved jlc** 2.86 mm to (215.9, 133.3)
Changed lines of the file:
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@@
   )
   (footprint "uni-footprints:jlc-tooling-hole" (layer "F.Cu")
-    (at 213.51875 131.7625)
+    (at 215.9 133.35)
     (fp_text reference "jlc**" (at 0 -0.5 unlocked) (layer "F.Fab")
       (effects (font (size 1 1) (thickness 0.15)))
@@
   )
   (footprint "uni-footprints:jlc-tooling-hole" (layer "F.Cu")
-    (at 46.83125 62.70625)
+    (at 30.1625 62.70625)
     (fp_text reference "jlc**" (at 0 -0.5 unlocked) (layer "F.Fab")
       (effects (font (size 1 1) (thickness 0.15)))
