File: unisplit_orthosteno.kicad_sch (KiCad schematic)
At the start: 58 parts, among them SW1 SW_SPST, U1 ProMicro

Commit message: add schematic
Parts:
- SW1: footprint uni-footprints:jumper-reversible -> Button_Switch_SMD:SW_SPST_TL3342
