File: Case/3dp-full-case/full-case-inner.kicad_pcb (KiCad board)
At the start: 2 copper layers, 260.6 x 89.2 mm, 6 parts

Commit message: fix fatal diode error
Other:
- board size 260.6 x 89.2 mm -> 248.6 x 77.2 mm
Changed lines of the file:
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@@
   )
   (gr_arc (start 30.1625 62.70625) (end 30.1625 59.825) (angle -90) (layer "Edge.Cuts") (width 0.05))
-  (gr_circle (center 256.38125 79.375) (end 259.38125 79.375) (layer "Edge.Cuts") (width 0.05) (fill none))
-  (gr_line (start 59.38125 134.14375) (end 59.53125 107.15625) (layer "Edge.Cuts") (width 0.05))
-  (gr_arc (start 273.05 62.70625) (end 281.93125 62.70625) (angle -90) (layer "Edge.Cuts") (width 0.05))
   (gr_arc (start 215.9 134.14375) (end 215.9 137.025) (angle -90) (layer "Edge.Cuts") (width 0.05))
   (gr_arc (start 273.05 96.04375) (end 273.05 98.925) (angle -90) (layer "Edge.Cuts") (width 0.05))
-  (gr_line (start 215.9 143.025) (end 68.2625 143.025) (layer "Edge.Cuts") (width 0.05))
   (gr_line (start 65.38125 134.14375) (end 65.38125 100.80625) (layer "Edge.Cuts") (width 0.05))
-  (gr_line (start 281.93125 62.70625) (end 281.93125 96.04375) (layer "Edge.Cuts") (width 0.05))
   (gr_line (start 30.1625 59.825) (end 273.05 59.825) (layer "Edge.Cuts") (width 0.05))
-  (gr_arc (start 30.1625 62.70625) (end 30.1625 53.825) (angle -90) (layer "Edge.Cuts") (width 0.05))
   (gr_line (start 218.78125 100.80625) (end 218.78125 134.14375) (layer "Edge.Cuts") (width 0.05))
   (gr_line (start 275.93125 62.70625) (end 275.93125 96.04375) (layer "Edge.Cuts") (width 0.05))
-  (gr_circle (center 180.18125 79.375) (end 183.18125 79.375) (layer "Edge.Cuts") (width 0.05) (fill none))
-  (gr_arc (start 30.1625 96.04375) (end 21.28125 96.04375) (angle -90) (layer "Edge.Cuts") (width 0.05))
   (gr_arc (start 220.6625 100.80625) (end 220.6625 98.925) (angle -90) (layer "Edge.Cuts") (width 0.05))
-  (gr_circle (center 199.23125 127) (end 202.23125 127) (layer "Edge.Cuts") (width 0.05) (fill none))
-  (gr_line (start 224.78125 134.14375) (end 224.78125 107.15625) (layer "Edge.Cuts") (width 0.05))
   (gr_line (start 27.28125 96.04375) (end 27.28125 62.70625) (layer "Edge.Cuts") (width 0.05))
   (gr_arc (start 63.5 100.80625) (end 65.38125 100.80625) (angle -90) (layer "Edge.Cuts") (width 0.05))
-  (gr_line (start 30.1625 53.825) (end 273.05 53.825) (layer "Edge.Cuts") (width 0.05))
-  (gr_arc (start 57.15 107.15625) (end 59.53125 107.15625) (angle -90) (layer "Edge.Cuts") (width 0.05))
-  (gr_arc (start 227.0125 107.15625) (end 227.0125 104.925) (angle -90) (layer "Edge.Cuts") (width 0.05))
-  (gr_line (start 21.28125 96.04375) (end 21.28125 62.70625) (layer "Edge.Cuts") (width 0.05))
-  (gr_circle (center 103.98125 79.375) (end 106.98125 79.375) (layer "Edge.Cuts") (width 0.05) (fill none))
   (gr_line (start 215.9 137.025) (end 68.2625 137.025) (layer "Edge.Cuts") (width 0.05))
   (gr_arc (start 68.2625 134.14375) (end 65.38125 134.14375) (angle -90) (layer "Edge.Cuts") (width 0.05))
-  (gr_arc (start 215.9 134.14375) (end 215.9 143.025) (angle -90) (layer "Edge.Cuts") (width 0.05))
-  (gr_circle (center 84.93125 127) (end 87.93125 127) (layer "Edge.Cuts") (width 0.05) (fill none))
-  (gr_circle (center 46.83125 79.375) (end 49.83125 79.375) (layer "Edge.Cuts") (width 0.05) (fill none))
-  (gr_arc (start 68.2625 134.14375) (end 59.38125 134.14375) (angle -90) (layer "Edge.Cuts") (width 0.05))
   (gr_arc (start 273.05 62.70625) (end 275.93125 62.70625) (angle -90) (layer "Edge.Cuts") (width 0.05))
-  (gr_line (start 57.15 104.775) (end 30.1625 104.925) (layer "Edge.Cuts") (width 0.05))
   (gr_arc (start 30.1625 96.04375) (end 27.28125 96.04375) (angle -90) (layer "Edge.Cuts") (width 0.05))
-  (gr_arc (start 273.05 96.04375) (end 273.05 104.925) (angle -90) (layer "Edge.Cuts") (width 0.05))
   (gr_line (start 63.5 98.925) (end 30.1625 98.925) (layer "Edge.Cuts") (width 0.05))
-  (gr_line (start 273.05 104.925) (end 227.0125 104.925) (layer "Edge.Cuts") (width 0.05))
   (gr_line (start 273.05 98.925) (end 220.6625 98.925) (layer "Edge.Cuts") (width 0.05))
 )
