File: Case/backplate/back-plate.kicad_pcb (KiCad board)
At the start: 2 copper layers, 247.6 x 76.2 mm, 7 parts

Commit message: gerbers and backplate
Parts:
- added REF**: jlc, uni-footprints:jlcjlcjlcjlc, B.Cu at (72.2, 134.9)
Changed lines of the file:
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@@
       (xy 3.496997 33.87885)) (layer "B.Mask") (width 0.01) (fill solid))
+  )
+  (footprint "uni-footprints:jlcjlcjlcjlc" (layer "B.Cu")
+    (at 72.23125 134.9375 180)
+    (fp_text reference "REF**" (at 0 0.5 unlocked) (layer "B.SilkS") hide
+      (effects (font (size 1 1) (thickness 0.15)) (justify mirror))
+    )
+    (fp_text value "jlc" (at 0 -1 unlocked) (layer "B.Fab") hide
+      (effects (font (size 1 1) (thickness 0.15)) (justify mirror))
+    )
+    (fp_text user "JLCJLCJLCJLC" (at 0 0) (layer "F.SilkS")
+      (effects (font (size 0.81 0.81) (thickness 0.15)))
+    )
   )
   (gr_line (start 27.78125 62.70625) (end 27.78125 96.04375) (layer "Edge.Cuts") (width 0.05))

Commit message: step file
Routing:
- added copper zone on F.Cu, net (none)
Changed lines of the file:
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@@
   (gr_arc (start 30.1625 96.04375) (end 27.78125 96.04375) (angle -90) (layer "Edge.Cuts") (width 0.05))
   (gr_arc (start 215.9 134.14375) (end 215.9 136.525) (angle -90) (layer "Edge.Cuts") (width 0.05))
-  (zone (net 0) (net_name "") (layer "B.Cu") (hatch edge 0.508)
+  (zone (net 0) (net_name "") (layers F&B.Cu) (hatch edge 0.508)
     (connect_pads (clearance 0.508))
     (min_thickness 0.254) (filled_areas_thickness no)

Commit message: caps update
Parts:
- REF**: moved to F.Cu
- REF** (x6), Ref**: moved to B.Cu
- moved REF** 209.6 mm to (256.4, 79.4), turned to 180 degrees
- moved REF** 209.6 mm to (46.8, 79.4), turned to 180 degrees
- moved REF** 133.3 mm to (218.3, 127.0), turned to 180 degrees
- moved REF** 95.2 mm to (199.2, 79.4), turned to 180 degrees
- moved REF** 95.2 mm to (104.0, 127.0), turned to 180 degrees
- moved Ref** 85.7 mm to (194.5, 90.1), turned to 180 degrees
- moved REF** 57.2 mm to (123.0, 79.4), turned to 180 degrees
- moved REF** 19.0 mm to (91.3, 134.9), turned to 0 degrees
Other:
- outline, holes or cut-outs redrawn
