File: Case/switchplate/MX-Choc/mx-choc-plate.kicad_pcb (KiCad board)
At the start: 2 copper layers, 247.6 x 76.2 mm, 6 parts

Commit message: plate stuff
Routing:
- removed copper zone on B.Cu, net (none)
- removed copper zone on F.Cu, net (none)
Changed lines of the file:
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@@
   (gr_arc (start 272.55625 76.2) (end 272.55625 76.7) (angle -90) (layer "Edge.Cuts") (width 0.2))
   (gr_arc (start 183.35625 63.200001) (end 183.35625 62.700001) (angle -90) (layer "Edge.Cuts") (width 0.2))
-  (zone (net 0) (net_name "") (layers F&B.Cu) (hatch edge 0.508)
-    (connect_pads (clearance 0.508))
-    (min_thickness 0.254) (filled_areas_thickness no)
-    (fill yes (thermal_gap 0.508) (thermal_bridge_width 0.508))
-    (polygon
-      (pts
-        (xy 275.43125 98.425)
-        (xy 219.075 99.21875)
-        (xy 218.28125 136.525)
-        (xy 65.88125 136.525)
-        (xy 65.0875 99.21875)
-        (xy 27.78125 98.425)
-        (xy 27.78125 60.325)
-        (xy 275.43125 60.325)
-      )
-    )
-  )
   (group "" (id 8a3d938a-9c9a-4343-b89d-fc526c764da3)
     (members

Commit message: add schematic
Parts:
- added REF**: MX_FMask-with-cutout, Keebio-Parts:MX_FMask-with-cutout, F.Cu at (265.9, 69.8)
- added REF**: MX_FMask-with-cutout, Keebio-Parts:MX_FMask-with-cutout, F.Cu at (208.8, 88.9)
- added REF**: MX_FMask-with-cutout, Keebio-Parts:MX_FMask-with-cutout, F.Cu at (189.7, 88.9)
- added REF**: MX_FMask-with-cutout, Keebio-Parts:MX_FMask-with-cutout, F.Cu at (227.8, 69.8)
- added REF**: MX_FMask-with-cutout, Keebio-Parts:MX_FMask-with-cutout, F.Cu at (75.4, 127.0)
- added REF**: MX_FMask-with-cutout, Keebio-Parts:MX_FMask-with-cutout, F.Cu at (75.4, 88.9)
- added REF**: MX_FMask-with-cutout, Keebio-Parts:MX_FMask-with-cutout, F.Cu at (56.4, 88.9)
- added REF**: MX_FMask-with-cutout, Keebio-Parts:MX_FMask-with-cutout, F.Cu at (189.7, 127.0)
- added REF**: MX_FMask-with-cutout, Keebio-Parts:MX_FMask-with-cutout, F.Cu at (170.7, 127.0)
- added REF**: MX_FMask-with-cutout, Keebio-Parts:MX_FMask-with-cutout, F.Cu at (56.4, 69.8)
- added REF**: MX_FMask-with-cutout, Keebio-Parts:MX_FMask-with-cutout, F.Cu at (246.9, 69.8)
- added REF**: MX_FMask-with-cutout, Keebio-Parts:MX_FMask-with-cutout, F.Cu at (265.9, 88.9)
- added REF**: MX_FMask-with-cutout, Keebio-Parts:MX_FMask-with-cutout, F.Cu at (75.4, 69.8)
- added REF**: MX_FMask-with-cutout, Keebio-Parts:MX_FMask-with-cutout, F.Cu at (246.9, 88.9)
- added REF**: MX_FMask-with-cutout, Keebio-Parts:MX_FMask-with-cutout, F.Cu at (189.7, 69.8)
- added REF**: MX_FMask-with-cutout, Keebio-Parts:MX_FMask-with-cutout, F.Cu at (208.8, 127.0)
- added REF**: MX_FMask-with-cutout, Keebio-Parts:MX_FMask-with-cutout, F.Cu at (227.8, 88.9)
- added REF**: MX_FMask-with-cutout, Keebio-Parts:MX_FMask-with-cutout, F.Cu at (208.8, 69.8)
- added REF**: MX_FMask-with-cutout, Keebio-Parts:MX_FMask-with-cutout, F.Cu at (113.5, 127.0)
- added REF**: MX_FMask-with-cutout, Keebio-Parts:MX_FMask-with-cutout, F.Cu at (94.5, 127.0)
- added REF**: MX_FMask-with-cutout, Keebio-Parts:MX_FMask-with-cutout, F.Cu at (37.3, 88.9)
- added REF**: MX_FMask-with-cutout, Keebio-Parts:MX_FMask-with-cutout, F.Cu at (113.5, 69.8)
- added REF**: MX_FMask-with-cutout, Keebio-Parts:MX_FMask-with-cutout, F.Cu at (37.3, 69.8)
- added REF**: MX_FMask-with-cutout, Keebio-Parts:MX_FMask-with-cutout, F.Cu at (94.5, 88.9)
- added REF**: MX_FMask-with-cutout, Keebio-Parts:MX_FMask-with-cutout, F.Cu at (170.7, 69.8)
- added REF**: MX_FMask-with-cutout, Keebio-Parts:MX_FMask-with-cutout, F.Cu at (94.5, 69.8)
- added REF**: MX_FMask-with-cutout, Keebio-Parts:MX_FMask-with-cutout, F.Cu at (113.5, 88.9)
- added REF**: MX_FMask-with-cutout, Keebio-Parts:MX_FMask-with-cutout, F.Cu at (170.7, 88.9)
- REF** (x6): value m4 -> m2; footprint MountingHole:MountingHole_4.3mm_M4_DIN965_Pad -> MountingHole:MountingHole_2.2mm_M2_DIN965_Pad
Other:
- outline, holes or cut-outs redrawn
